File: hardware/board/frost.kicad_pcb (KiCad board)
At the start: 2 copper layers, 90 x 55 mm, 288 parts, among them CN1 AXT530124_C2924271, Q1 WPM3407-3/TR, Q2 SS8050, Q3 WPM2015-3/TR_C7472861, Q4 WPM2015-3/TR_C7472861, Q5 SS8050, U1 RK3568, U10 SY8088AAC, U11 RK860-0, U12 SY7208ABC, U13 FTC252012SR24MBCA, U14 ESD5311X, U15 ESD5311X, U16 ESD5311X, U17 ESD5311X, U18 SY6280AAC, U19 ESD5311X, U2 K4UCE3Q4AB-MGCL, U20 ESD5311X, U21 ESD5311X, U22 ESD5311X, U23 ESD5311X, U24 ESD5311X, U25 ESD5311X, U26 LP3983SAB5F-08, U3 KLMBG2JETD-B041_C5821038, U4 RK809-5, U5 AP6256, U6 TMUXHS4212RKSR, U7 FUSB302BMPX, U8 BQ25890RTWR, U9 S2B-PH-K-S(LF)(SN), X1 24 MHz, X2 Q13FC1350000400

Commit message: start of ethernet
Parts:
- added C122: 47uF X5R 6.3V, Capacitor_SMD:C_0805_2012Metric, F.Cu at (79.3, 78.0)
- added C147: 1uF X5R 10V, Capacitor_SMD:C_0402_1005Metric, F.Cu at (128.1, 66.7)
- added C148: 10uF X5R 10V, Capacitor_SMD:C_0603_1608Metric, F.Cu at (58.8, 83.2)
- added C149: 100nF X5R 10V, Capacitor_SMD:C_0402_1005Metric, F.Cu at (70.3, 89.9)
- added C150: 2.2uF X5R 50V, Capacitor_SMD:C_0805_2012Metric, F.Cu at (71.7, 86.8)
- added C151: 10uF X5R 6.3V, Capacitor_SMD:C_0603_1608Metric, F.Cu at (58.8, 85.7)
- added C152: 100nF X5R 10V, Capacitor_SMD:C_0402_1005Metric, F.Cu at (70.3, 91.9)
- added C153: 10uF X5R 6.3V, Capacitor_SMD:C_0603_1608Metric, F.Cu at (58.8, 88.2)
- added C154: 4.7uF X5R 6.3V, Capacitor_SMD:C_0603_1608Metric, F.Cu at (58.8, 90.7)
- added C155: 100nF X5R 10V, Capacitor_SMD:C_0402_1005Metric, F.Cu at (70.3, 93.9)
- added C156: 22uF X5R 10V, Capacitor_SMD:C_0805_2012Metric, F.Cu at (132.9, 33.3)
- added C157: 100nF X5R 10V, Capacitor_SMD:C_0402_1005Metric, F.Cu at (130.8, 39.7)
- added C158: 20pF C0G 50V, Capacitor_SMD:C_0402_1005Metric, F.Cu at (130.8, 41.7)
- added C159: 20pF C0G 50V, Capacitor_SMD:C_0402_1005Metric, F.Cu at (130.8, 43.7)
- added C160: 4.7uF X5R 10V, Capacitor_SMD:C_0603_1608Metric, F.Cu at (111.2, 25.1)
- added C161: 4.7uF X5R 10V, Capacitor_SMD:C_0603_1608Metric, F.Cu at (111.2, 27.6)
- added C162: 100nF X5R 10V, Capacitor_SMD:C_0402_1005Metric, F.Cu at (130.8, 45.7)
- added C163: 4.7uF X5R 10V, Capacitor_SMD:C_0603_1608Metric, F.Cu at (111.2, 30.2)
- added C164: 100pF X5R 25V, Capacitor_SMD:C_0201_0603Metric, F.Cu at (128.2, 39.6)
- added C165: 100pF X5R 25V, Capacitor_SMD:C_0201_0603Metric, F.Cu at (128.2, 41.4)
- added C166: 100nF X5R 10V, Capacitor_SMD:C_0201_0603Metric, F.Cu at (128.2, 43.1)
- added C167: 100nF X5R 10V, Capacitor_SMD:C_0201_0603Metric, F.Cu at (128.2, 44.9)
- added C168: 100nF X5R 10V, Capacitor_SMD:C_0201_0603Metric, F.Cu at (128.2, 46.6)
- added C169: 100nF X5R 10V, Capacitor_SMD:C_0201_0603Metric, F.Cu at (128.2, 48.4)
- added C170: DNP, Capacitor_SMD:C_0402_1005Metric, F.Cu at (130.8, 47.6)
- added C171: DNP, Capacitor_SMD:C_0402_1005Metric, F.Cu at (133.7, 39.7)
- added C172: DNP, Capacitor_SMD:C_0402_1005Metric, F.Cu at (133.7, 41.7)
- added C173: DNP, Capacitor_SMD:C_0402_1005Metric, F.Cu at (133.7, 43.7)
- added C174: DNP, Capacitor_SMD:C_0402_1005Metric, F.Cu at (133.7, 45.7)
- added C175: DNP, Capacitor_SMD:C_0402_1005Metric, F.Cu at (133.7, 47.6)
- added C176: 10pF C0G 50V, Capacitor_SMD:C_0201_0603Metric, F.Cu at (128.2, 50.1)
- added C177: 20pF C0G 50V, Capacitor_SMD:C_0402_1005Metric, F.Cu at (99.3, 24.9)
- added C178: 20pF C0G 50V, Capacitor_SMD:C_0402_1005Metric, F.Cu at (99.3, 26.8)
- added C179: 100nF X5R 10V, Capacitor_SMD:C_0402_1005Metric, F.Cu at (99.3, 28.8)
- added C180: 100nF X5R 10V, Capacitor_SMD:C_0402_1005Metric, F.Cu at (99.3, 30.8)
- added C181: 4.7uF X5R 10V, Capacitor_SMD:C_0603_1608Metric, F.Cu at (97.6, 61.1)
- added C182: 100nF X5R 10V, Capacitor_SMD:C_0402_1005Metric, F.Cu at (99.3, 32.7)
- added C183: 100nF X5R 10V, Capacitor_SMD:C_0402_1005Metric, F.Cu at (102.2, 24.9)
- added C184: 100nF X5R 10V, Capacitor_SMD:C_0402_1005Metric, F.Cu at (102.2, 26.8)
- added C185: 100nF X5R 10V, Capacitor_SMD:C_0402_1005Metric, F.Cu at (102.2, 28.8)
- added C186: 4.7uF X5R 10V, Capacitor_SMD:C_0603_1608Metric, F.Cu at (97.6, 63.6)
- added C187: 100nF X5R 10V, Capacitor_SMD:C_0402_1005Metric, F.Cu at (102.2, 30.8)
- added C188: 1uF X5R 10V, Capacitor_SMD:C_0402_1005Metric, F.Cu at (102.2, 32.7)
- added C189: 4.7uF X5R 10V, Capacitor_SMD:C_0603_1608Metric, F.Cu at (97.6, 66.1)
- added C190: 100nF X5R 10V, Capacitor_SMD:C_0402_1005Metric, F.Cu at (105.0, 24.9)
- added C191: 100nF X5R 10V, Capacitor_SMD:C_0402_1005Metric, F.Cu at (105.0, 26.8)
- added C192: 4.7uF X5R 10V, Capacitor_SMD:C_0603_1608Metric, F.Cu at (97.6, 68.6)
- added C193: 100nF X5R 10V, Capacitor_SMD:C_0402_1005Metric, F.Cu at (105.0, 28.8)
- added D12: ESD5344D, lcsc:DFN2510-10_L2.5-W1.0-P0.50-BL, F.Cu at (120.6, 67.0)
- added D13: ESD5344D, lcsc:DFN2510-10_L2.5-W1.0-P0.50-BL, F.Cu at (120.6, 69.9)
- added D14: B5819WS_C916992, lcsc:SOD-323_L1.7-W1.3-LS2.5-RD, F.Cu at (124.6, 67.0)
- added D15: B5819WS_C916992, lcsc:SOD-323_L1.7-W1.3-LS2.5-RD, F.Cu at (124.6, 69.5)
- added D16: SS34, Diode_SMD:D_SMA, F.Cu at (64.9, 91.2)
- added D17: LED GREEN, LED_SMD:LED_0603_1608Metric, F.Cu at (101.6, 69.6)
- added D18: LED YELLOW, LED_SMD:LED_0603_1608Metric, F.Cu at (101.6, 72.2)
- added FPC1: HC-FPC-03-09-31RLTAG, lcsc:FPC-SMD_31P-P0.30_HC-FPC-03-09-31RLTAG, F.Cu at (63.2, 78.9)
- added J1: HDMI_A, Connector_Video:HDMI_A_Amphenol_10029449-x01xLF_Horizontal, F.Cu at (121.9, 60.2)
- added Q6: 2SK3018_C194460, lcsc:SOT-323-3_L2.0-W1.3-P1.30-LS2.1-BR, F.Cu at (114.0, 67.4)
- added Q7: 2SK3018_C194460, lcsc:SOT-323-3_L2.0-W1.3-P1.30-LS2.1-BR, F.Cu at (114.0, 70.8)
- added Q8: 2SK3018_C194460, lcsc:SOT-323-3_L2.0-W1.3-P1.30-LS2.1-BR, F.Cu at (114.0, 74.2)
- added R100: 120R 5%, Resistor_SMD:R_0402_1005Metric, F.Cu at (97.0, 44.9)
- added R101: 100R 5%, Resistor_SMD:R_0402_1005Metric, F.Cu at (97.0, 46.9)
- added R102: 2.49K 1%, Resistor_SMD:R_0402_1005Metric, F.Cu at (97.0, 48.9)
- added R103: 0R 5%, Resistor_SMD:R_0402_1005Metric, F.Cu at (97.0, 50.9)
- added R104: 0R 5%, Resistor_SMD:R_0402_1005Metric, F.Cu at (97.0, 52.8)
- added R105: 1.8K 5%, Resistor_SMD:R_0402_1005Metric, F.Cu at (97.0, 54.8)
- added R106: 22R 5%, Resistor_SMD:R_0402_1005Metric, F.Cu at (97.0, 56.8)
- added R107: 22R 5%, Resistor_SMD:R_0402_1005Metric, F.Cu at (97.0, 58.8)
- added R108: 22R 5%, Resistor_SMD:R_0402_1005Metric, F.Cu at (99.9, 44.9)
- added R109: 22R 5%, Resistor_SMD:R_0402_1005Metric, F.Cu at (99.9, 46.9)
- added R110: 22R 5%, Resistor_SMD:R_0402_1005Metric, F.Cu at (99.9, 48.9)
- added R111: 22R 5%, Resistor_SMD:R_0402_1005Metric, F.Cu at (99.9, 50.9)
- added R112: 4.7K 5%, Resistor_SMD:R_0402_1005Metric, F.Cu at (99.9, 52.8)
- added R113: 4.7K 5%, Resistor_SMD:R_0402_1005Metric, F.Cu at (99.9, 54.8)
- added R114: 4.7K 5%, Resistor_SMD:R_0402_1005Metric, F.Cu at (99.9, 56.8)
- added R115: 4.7K 5%, Resistor_SMD:R_0402_1005Metric, F.Cu at (99.9, 58.8)
- added R116: 4.7K 5%, Resistor_SMD:R_0402_1005Metric, F.Cu at (102.8, 44.9)
- added R117: 4.7K 5%, Resistor_SMD:R_0402_1005Metric, F.Cu at (102.8, 46.9)
- added R118: 4.7K 5%, Resistor_SMD:R_0402_1005Metric, F.Cu at (102.8, 48.9)
- added R119: 4.7K 5%, Resistor_SMD:R_0402_1005Metric, F.Cu at (102.8, 50.9)
- added R120: 4.7K 5%, Resistor_SMD:R_0402_1005Metric, F.Cu at (102.8, 52.8)
- added R121: 4.7K 5%, Resistor_SMD:R_0402_1005Metric, F.Cu at (102.8, 54.8)
- added R122: 4.7K 5%, Resistor_SMD:R_0402_1005Metric, F.Cu at (102.8, 56.8)
- added R123: 4.7K 5%, Resistor_SMD:R_0402_1005Metric, F.Cu at (102.8, 58.8)
- added R124: 4.7K 5%, Resistor_SMD:R_0402_1005Metric, F.Cu at (105.8, 44.9)
- added R125: 4.7K 5%, Resistor_SMD:R_0402_1005Metric, F.Cu at (105.8, 46.9)
- added R126: 4.7K 5%, Resistor_SMD:R_0402_1005Metric, F.Cu at (105.8, 48.9)
- added R127: 510R 5%, Resistor_SMD:R_0402_1005Metric, F.Cu at (105.8, 50.9)
- added R128: 0R 5%, Resistor_SMD:R_0402_1005Metric, F.Cu at (105.8, 52.8)
- added R129: 510R 5%, Resistor_SMD:R_0402_1005Metric, F.Cu at (105.8, 54.8)
- added R130: 0R 5%, Resistor_SMD:R_0402_1005Metric, F.Cu at (105.8, 56.8)
- added R82: 1.8K 5%, Resistor_SMD:R_0402_1005Metric, F.Cu at (110.7, 54.2)
- added R83: 10K 5%, Resistor_SMD:R_0402_1005Metric, F.Cu at (110.7, 56.2)
- added R84: 10K 5%, Resistor_SMD:R_0402_1005Metric, F.Cu at (110.7, 58.2)
- added R85: 1.8K 5%, Resistor_SMD:R_0402_1005Metric, F.Cu at (110.7, 60.2)
- added R86: 27K 5%, Resistor_SMD:R_0402_1005Metric, F.Cu at (110.7, 62.1)
- added R87: 1K 5%, Resistor_SMD:R_0402_1005Metric, F.Cu at (110.7, 64.1)
- added R88: 100K 5%, Resistor_SMD:R_0402_1005Metric, F.Cu at (110.7, 66.1)
- added R89: 0R 5%, Resistor_SMD:R_0402_1005Metric, F.Cu at (73.2, 89.9)
- added R90: 100K 5%, Resistor_SMD:R_0402_1005Metric, F.Cu at (73.2, 91.9)
- added R91: 5.1R 5%, Resistor_SMD:R_1206_3216Metric, F.Cu at (72.3, 83.6)
- added R92: 22R 5%, Resistor_SMD:R_0402_1005Metric, F.Cu at (132.1, 24.9)
- added R93: 22R 5%, Resistor_SMD:R_0402_1005Metric, F.Cu at (132.1, 26.9)
- added R94: 0R 5%, Resistor_SMD:R_0402_1005Metric, F.Cu at (132.1, 28.9)
- added R95: 0R 5%, Resistor_SMD:R_0603_1608Metric, F.Cu at (111.2, 32.7)
- added R96: 0R 5%, Resistor_SMD:R_0603_1608Metric, F.Cu at (111.2, 35.2)
- added R97: 0R 5%, Resistor_SMD:R_0603_1608Metric, F.Cu at (111.2, 37.7)
- added R98: 10K 5%, Resistor_SMD:R_0402_1005Metric, F.Cu at (132.1, 30.8)
- added R99: 0R 5%, Resistor_SMD:R_0603_1608Metric, F.Cu at (111.2, 40.2)
- added RF1: BWIPX-1-001E, lcsc:IPEX-SMD_BWIPX-1-001E, F.Cu at (115.0, 41.3)
- added RF2: BWIPX-1-001E, lcsc:IPEX-SMD_BWIPX-1-001E, F.Cu at (119.6, 41.3)
- added RF3: BWIPX-1-001E, lcsc:IPEX-SMD_BWIPX-1-001E, F.Cu at (124.1, 41.3)
- added RJ1: R-RJ45R08P-C000, lcsc:RJ45-TH_R-RJ45R08P-C000, F.Cu at (66.7, 29.1)
- added RJ2: R-RJ45R08P-C000, lcsc:RJ45-TH_R-RJ45R08P-C000, F.Cu at (66.7, 46.2)
- added RJ3: R-RJ45R10P-B000, lcsc:RJ45-TH_R-RJ45R10P-B000, F.Cu at (86.1, 55.3)
- added RJ4: HC-RJ45-5JA-1-5, lcsc:RJ45-TH_HC-RJ45-5JA-1-5, F.Cu at (65.4, 63.2)
- added RJ5: 2-406549-1, lcsc:RJ45-TH_2-406549-1, F.Cu at (87.2, 30.7)
- added U27: 5054133410_C6422029, lcsc:CONN-SMD_5054133410, F.Cu at (206.2, 98.0)
- added U28: ESD5341N, lcsc:DFN1006-2L-RD, F.Cu at (117.3, 66.7)
- added U29: ESD5341N, lcsc:DFN1006-2L-RD, F.Cu at (117.3, 68.8)
- added U30: ESD5341N, lcsc:DFN1006-2L-RD, F.Cu at (117.3, 70.9)
- added U31: ESD5341N, lcsc:DFN1006-2L-RD, F.Cu at (117.3, 73.0)
- added U32: SY7203DBC, lcsc:DFN-10_L3.0-W3.0-P0.50-BL-EP2.4, F.Cu at (71.7, 78.8)
- added U33: CY54-4.7UH, lcsc:IND-SMD_L5.8-W5.2, F.Cu at (65.2, 85.5)
- added U34: AP6275PR3, lcsc:WIRELM-SMD_AMPAK_AP6275P, F.Cu at (122.3, 31.3)
- added U35: TFM252012ALVA2R2MTAA, lcsc:L1008, F.Cu at (116.1, 49.3)
- added U36: RTL8211F-CG, lcsc:WQFN-40_L5.0-W5.0-P0.4-BL-EP, F.Cu at (101.3, 37.1)
- added U37: TFM252012ALVA2R2MTAA, lcsc:L1008, F.Cu at (102.4, 61.7)
- added U5: TFM252012ALVA2R2MTAA, lcsc:L1008, F.Cu at (116.1, 45.6)
- added X3: S3237400121040, lcsc:CRYSTAL-SMD_4P-L3.2-W2.5-BL, F.Cu at (121.7, 46.0)
- added X4: X322525MOB4SI, lcsc:CRYSTAL-SMD_4P-L3.2-W2.5-BL, F.Cu at (102.4, 65.8)
Connections:
- C48 pad 1: VCC_1V8 -> VCCA1V8_IMAGE
- FB3 pad 2: VCC_1V8 -> VCCA1V8_IMAGE

Commit message: finish ethernet
Parts:
- removed the C122 at (204.0, 74.3)
- removed CN1: AXT530124_C2924271, lcsc:CONN-SMD_30P-P0.40_AXT530124
- removed D17: LED GREEN, LED_SMD:LED_0603_1608Metric
- removed D18: LED YELLOW, LED_SMD:LED_0603_1608Metric
- removed R129: 510R 5%, Resistor_SMD:R_0402_1005Metric
- removed RJ2: R-RJ45R08P-C000, lcsc:RJ45-TH_R-RJ45R08P-C000
- removed RJ3: R-RJ45R10P-B000, lcsc:RJ45-TH_R-RJ45R10P-B000
- removed RJ4: HC-RJ45-5JA-1-5, lcsc:RJ45-TH_HC-RJ45-5JA-1-5
- removed RJ5: 2-406549-1, lcsc:RJ45-TH_2-406549-1
- removed the U5 at (170.3, 108.8)
- added C194: 10nF X5R 25V, Capacitor_SMD:C_0402_1005Metric, F.Cu at (111.9, 99.1)
- added C195: 10nF X5R 25V, Capacitor_SMD:C_0402_1005Metric, F.Cu at (111.9, 101.0)
- added C196: 10nF X5R 25V, Capacitor_SMD:C_0402_1005Metric, F.Cu at (111.9, 103.0)
- added C197: 10nF X5R 25V, Capacitor_SMD:C_0402_1005Metric, F.Cu at (111.9, 105.0)
- added FB11: 120@100MHz 25% 2A, Inductor_SMD:L_0603_1608Metric, F.Cu at (37.3, 128.6)
- added R131: 0R 5%, Resistor_SMD:R_0402_1005Metric, F.Cu at (103.2, 101.1)
- added R132: 0R 5%, Resistor_SMD:R_0402_1005Metric, F.Cu at (103.2, 103.1)
- added R133: 0R 5%, Resistor_SMD:R_0402_1005Metric, F.Cu at (103.2, 105.1)
- added R134: 0R 5%, Resistor_SMD:R_0402_1005Metric, F.Cu at (103.2, 107.0)
- added R135: 0R 5%, Resistor_SMD:R_0402_1005Metric, F.Cu at (106.1, 99.1)
- added R136: 0R 5%, Resistor_SMD:R_0402_1005Metric, F.Cu at (106.1, 101.1)
- added R137: 0R 5%, Resistor_SMD:R_0402_1005Metric, F.Cu at (106.1, 103.1)
- added R138: 0R 5%, Resistor_SMD:R_0402_1005Metric, F.Cu at (106.1, 105.1)
- added U38: ESD5451N_C5261080, lcsc:DFN1006-2L-BI, F.Cu at (36.7, 113.1)
- added U39: ESD5451N_C5261080, lcsc:DFN1006-2L-BI, F.Cu at (36.7, 115.0)
- added U40: ESD5451N_C5261080, lcsc:DFN1006-2L-BI, F.Cu at (36.7, 116.9)
- added U41: ESD5451N_C5261080, lcsc:DFN1006-2L-BI, F.Cu at (36.7, 118.8)
- added U42: ESD5451N_C5261080, lcsc:DFN1006-2L-BI, F.Cu at (36.7, 120.7)
- added U43: ESD5451N_C5261080, lcsc:DFN1006-2L-BI, F.Cu at (36.7, 122.6)
- added U44: ESD5451N_C5261080, lcsc:DFN1006-2L-BI, F.Cu at (36.7, 124.5)
- added U45: ESD5451N_C5261080, lcsc:DFN1006-2L-BI, F.Cu at (36.7, 126.4)
- R128: value 0R 5% -> 510R 5%
- RJ1: value R-RJ45R08P-C000 -> HY911130A; footprint lcsc:RJ45-TH_R-RJ45R08P-C000 -> lcsc:RJ45-TH_10P-P2.54-S2.54_L16.1-W21.4_HY911130A
- moved RJ1 100.8 mm to (25.8, 121.2)
- moved R128 46.3 mm to (103.2, 99.1)
- moved D12 14.4 mm to (134.7, 69.5)
Connections:
- R127 pad 1: VCC3V3_PHY0 -> /Ethernet/PHY0_LED1_N
- R127 pad 2: Net-(D18-A) -> /Ethernet/PHY0_LED1/CFG_LDO0
- R128 pad 1: /Ethernet/PHY0_LED2/CFG_LDO1 -> /Ethernet/PHY0_LED2_N
- R128 pad 2: Net-(D18-K) -> /Ethernet/PHY0_LED2/CFG_LDO1
- RJ1 pad 1: unconnected-(RJ1-Pad1) -> Net-(C194-Pad1)
- RJ1 pad 10: unconnected-(RJ1-L--Pad10) -> (no net)
- RJ1 pad 11: unconnected-(RJ1-R+-Pad11) -> /Ethernet/PHY0_LED1_N
- RJ1 pad 12: unconnected-(RJ1-R--Pad12) -> GND
- RJ1 pad 13: unconnected-(RJ1-S-Pad13) -> /Ethernet/PHY0_LED2_N
- RJ1 pad 14: unconnected-(RJ1-S-Pad14) -> VCC3V3_PHY0
- RJ1 pad 2: unconnected-(RJ1-Pad2) -> GND
- RJ1 pad 3: unconnected-(RJ1-Pad3) -> Net-(R132-Pad2)
- RJ1 pad 4: unconnected-(RJ1-Pad4) -> Net-(R133-Pad2)
- RJ1 pad 5: unconnected-(RJ1-Pad5) -> Net-(R134-Pad2)
- RJ1 pad 6: unconnected-(RJ1-Pad6) -> Net-(R135-Pad2)
- RJ1 pad 7: unconnected-(RJ1-Pad7) -> Net-(R136-Pad2)
- RJ1 pad 8: unconnected-(RJ1-Pad8) -> Net-(R137-Pad2)
- RJ1 pad 9: unconnected-(RJ1-L+-Pad9) -> (no net)

Commit message: aaa
Connections:
- net /Ethernet/PHY0_LED1_N renamed /Ethernet/PHY0_LED1_P
- R103 pad 2: PHY0_LED0/CFG_EXT -> GMAC0_INT/PMEB_GPIO3_C0
- R104 pad 1: GMAC0_MCLKINOUT -> GMAC0_RSTn_GPIO3_B0
- R112 pad 1: PHY0_LED0/CFG_EXT -> /Ethernet/PHY0_LED0/CFG_EXT
- R113 pad 2: PHY0_LED0/CFG_EXT -> /Ethernet/PHY0_LED0/CFG_EXT
- U36 pad 32: PHY0_LED0/CFG_EXT -> /Ethernet/PHY0_LED0/CFG_EXT
Changed lines of the file:
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@@
 	(net 1028 "/Ethernet/RSET0")
 	(net 1029 "Net-(U36-INTB{slash}PMEB)")
-	(net 1030 "PHY0_LED0{slash}CFG_EXT")
+	(net 1030 "GMAC0_INT{slash}PMEB_GPIO3_C0")
 	(net 1031 "GMAC0_MDIO")
 	(net 1032 "/Ethernet/PHY0_RXD0{slash}RXDLY")
@@
 	(net 1089 "GMAC0_TXD1")
 	(net 1090 "Net-(FB11-Pad1)")
-	(net 1091 "/Ethernet/PHY0_LED1_N")
+	(net 1091 "GMAC0_RSTn_GPIO3_B0")
 	(net 1092 "Net-(RJ1-9)")
+	(net 1093 "/Ethernet/PHY0_LED0{slash}CFG_EXT")
+	(net 1094 "/Ethernet/PHY0_LED1_P")
 	(footprint "Capacitor_SMD:C_0402_1005Metric"
 		(layer "F.Cu")
@@
 			(layers "F.Cu" "F.Mask" "F.Paste")
 			(roundrect_rratio 0.25)
-			(net 1030 "PHY0_LED0{slash}CFG_EXT")
+			(net 1093 "/Ethernet/PHY0_LED0{slash}CFG_EXT")
 			(pintype "passive")
 		)
@@
 			(layers "F.Cu" "F.Mask" "F.Paste")
 			(roundrect_rratio 0.25)
-			(net 1091 "/Ethernet/PHY0_LED1_N")
+			(net 1094 "/Ethernet/PHY0_LED1_P")
 			(pintype "passive")
 		)
@@
 			(layers "F.Cu" "F.Mask" "F.Paste")
 			(roundrect_rratio 0.25)
-			(net 1030 "PHY0_LED0{slash}CFG_EXT")
+			(net 1093 "/Ethernet/PHY0_LED0{slash}CFG_EXT")
 			(pintype "passive")
 		)
@@
 			(layers "F.Cu" "F.Mask" "F.Paste")
 			(roundrect_rratio 0.25)
-			(net 1026 "GMAC0_MCLKINOUT")
+			(net 1091 "GMAC0_RSTn_GPIO3_B0")
 			(pintype "passive")
 		)
@@
 			(size 0.2 0.8)
 			(layers "F.Cu" "F.Mask" "F.Paste")
-			(net 1030 "PHY0_LED0{slash}CFG_EXT")
+			(net 1093 "/Ethernet/PHY0_LED0{slash}CFG_EXT")
 			(pinfunction "CFG_EXT/LED0")
 			(pintype "unspecified")
@@
 			(layers "*.Cu" "*.Mask")
 			(remove_unused_layers no)
-			(net 1091 "/Ethernet/PHY0_LED1_N")
+			(net 1094 "/Ethernet/PHY0_LED1_P")
 			(pinfunction "11")
 			(pintype "unspecified")
@@
 			(layers "F.Cu" "F.Mask" "F.Paste")
 			(roundrect_rratio 0.25)
-			(net 1030 "PHY0_LED0{slash}CFG_EXT")
+			(net 1030 "GMAC0_INT{slash}PMEB_GPIO3_C0")
 			(pintype "passive")
 		)
