File: hardware/board/frost.kicad_pcb (KiCad board)
At the start: 2 copper layers, 90 x 55 mm, 565 parts, among them CN1 PJ-393 8PJ, CN2 1-2199230-5, CN2 35RAPC4BH3, J1 HDMI_A, Q1 WPM3407-3/TR, Q2 SS8050, Q3 WPM2015-3/TR_C7472861, Q4 WPM2015-3/TR_C7472861, Q5 SS8050, Q6 2SK3018_C194460, Q7 2SK3018_C194460, Q8 2SK3018_C194460, U1 RK3568, U10 SY8088AAC, U11 RK860-0, U12 SY7208ABC, U13 FTC252012SR24MBCA, U14 ESD5311X, U15 ESD5311X, U16 ESD5311X, U17 ESD5311X, U18 SY6280AAC, U19 ESD5311X, U2 K4UCE3Q4AB-MGCL, U20 ESD5311X, U21 ESD5311X, U22 ESD5311X, U23 ESD5311X, U24 ESD5311X, U25 ESD5311X, U26 LP3983SAB5F-08, U27 5054133410_C6422029, U28 ESD5341N, U29 ESD5341N, U3 KLMBG2JETD-B041_C5821038, U30 ESD5341N, U31 ESD5341N, U32 SY7203DBC, U33 CY54-4.7UH, U34 AP6275PR3, U35 TFM252012ALVA2R2MTAA, U36 RTL8211F-CG, U37 TFM252012ALVA2R2MTAA, U38 ESD5451N_C5261080, U39 ESD5451N_C5261080, U4 RK809-5, U40 ESD5451N_C5261080, U41 ESD5451N_C5261080, U42 ESD5451N_C5261080, U43 ESD5451N_C5261080, U44 ESD5451N_C5261080, U45 ESD5451N_C5261080, U46 ESD5451N_C5261080, U47 ESD5451N_C5261080, U48 ESD5451N_C5261080, U49 ESD5451N_C5261080, U5 TFM252012ALVA2R2MTAA, U6 TMUXHS4212RKSR, U7 FUSB302BMPX, U8 BQ25890RTWR, U9 S2B-PH-K-S(LF)(SN), X1 24 MHz, X2 Q13FC1350000400, X3 S3237400121040, X4 X322525MOB4SI

Commit message: aaaa
Parts:
- added C301: 22uF X5R 6.3V, Capacitor_SMD:C_0603_1608Metric, F.Cu at (250.8, 41.3)
- added C302: 100nF X5R 10V, Capacitor_SMD:C_0402_1005Metric, F.Cu at (252.2, 53.0)
- added C303: 22uF X5R 6.3V, Capacitor_SMD:C_0603_1608Metric, F.Cu at (250.8, 43.8)
- added C304: 100nF X5R 10V, Capacitor_SMD:C_0402_1005Metric, F.Cu at (252.2, 55.0)
- added C305: 18pF C0G 50V, Capacitor_SMD:C_0402_1005Metric, F.Cu at (252.2, 56.9)
- added C306: 18pF C0G 50V, Capacitor_SMD:C_0402_1005Metric, F.Cu at (252.2, 58.9)
- added C307: 1uF X5R 10V, Capacitor_SMD:C_0402_1005Metric, F.Cu at (255.1, 53.0)
- added C308: 100nF X5R 10V, Capacitor_SMD:C_0402_1005Metric, F.Cu at (255.1, 55.0)
- added C309: 1uF X5R 10V, Capacitor_SMD:C_0402_1005Metric, F.Cu at (255.1, 56.9)
- added C310: 100nF X5R 10V, Capacitor_SMD:C_0402_1005Metric, F.Cu at (255.1, 58.9)
- added C311: 4.7F X5R 6.3V, Capacitor_SMD:C_0402_1005Metric, F.Cu at (257.9, 53.0)
- added C312: 1uF X5R 10V, Capacitor_SMD:C_0402_1005Metric, F.Cu at (257.9, 55.0)
- added C313: 100nF X5R 10V, Capacitor_SMD:C_0402_1005Metric, F.Cu at (257.9, 56.9)
- added C314: 4.7F X5R 6.3V, Capacitor_SMD:C_0402_1005Metric, F.Cu at (257.9, 58.9)
- added C315: 10uF X5R 10V, Capacitor_SMD:C_0603_1608Metric, F.Cu at (250.8, 46.4)
- added C316: 100nF X5R 10V, Capacitor_SMD:C_0402_1005Metric, F.Cu at (260.8, 53.0)
- added C317: 100nF X5R 10V, Capacitor_SMD:C_0402_1005Metric, F.Cu at (260.8, 55.0)
- added C318: 22pF C0G 50V, Capacitor_SMD:C_0402_1005Metric, F.Cu at (260.8, 56.9)
- added C319: 10uF X5R 6.3V, Capacitor_SMD:C_0603_1608Metric, F.Cu at (250.8, 48.9)
- added C320: 22pF C0G 50V, Capacitor_SMD:CP_Elec_6.3x5.9, F.Cu at (245.4, 56.1)
- added C321: 100nF X5R 10V, Capacitor_SMD:C_0402_1005Metric, F.Cu at (260.8, 58.9)
- added L11: LVF404026-2R2M-N, lcsc:IND-SMD_L4.0-W4.0, F.Cu at (253.7, 62.6)
- added R152: 22R 5%, Resistor_SMD:R_0402_1005Metric, F.Cu at (241.6, 41.1)
- added R153: 22R 5%, Resistor_SMD:R_0402_1005Metric, F.Cu at (241.6, 43.1)
- added R154: 22R 5%, Resistor_SMD:R_0402_1005Metric, F.Cu at (241.6, 45.0)
- added R155: 22R 5%, Resistor_SMD:R_0402_1005Metric, F.Cu at (241.6, 47.0)
- added R156: 2.2R 5%, Resistor_SMD:R_0402_1005Metric, F.Cu at (241.6, 49.0)
- added R157: 33R 5%, Resistor_SMD:R_0201_0603Metric, F.Cu at (238.9, 41.0)
- added R158: 33R 5%, Resistor_SMD:R_0201_0603Metric, F.Cu at (238.9, 42.7)
- added R159: 49.9R 1%, Resistor_SMD:R_0201_0603Metric, F.Cu at (238.9, 44.5)
- added R160: 49.9R 1%, Resistor_SMD:R_0201_0603Metric, F.Cu at (238.9, 46.2)
- added R161: 33R 5%, Resistor_SMD:R_0201_0603Metric, F.Cu at (238.9, 48.0)
- added R162: 33R 5%, Resistor_SMD:R_0201_0603Metric, F.Cu at (238.9, 49.7)
- added R163: 49.9R 1%, Resistor_SMD:R_0201_0603Metric, F.Cu at (238.9, 51.5)
- added R164: 49.9R 1%, Resistor_SMD:R_0201_0603Metric, F.Cu at (238.9, 53.2)
- added R165: 470R 1%, Resistor_SMD:R_0402_1005Metric, F.Cu at (241.6, 51.0)
- added R166: 10K 5%, Resistor_SMD:R_0402_1005Metric, F.Cu at (244.5, 41.1)
- added R167: 10K 5%, Resistor_SMD:R_0402_1005Metric, F.Cu at (244.5, 43.1)
- added R168: 10K 5%, Resistor_SMD:R_0402_1005Metric, F.Cu at (244.5, 45.0)
- added R169: 10K 5%, Resistor_SMD:R_0402_1005Metric, F.Cu at (244.5, 47.0)
- added R170: 10K 5%, Resistor_SMD:R_0402_1005Metric, F.Cu at (244.5, 49.0)
- added R171: 10K 5%, Resistor_SMD:R_0402_1005Metric, F.Cu at (244.5, 51.0)
- added R172: 10K 5%, Resistor_SMD:R_0402_1005Metric, F.Cu at (247.4, 41.1)
- added R173: 470R 1%, Resistor_SMD:R_0402_1005Metric, F.Cu at (247.4, 43.1)
- added R174: 10K 5%, Resistor_SMD:R_0402_1005Metric, F.Cu at (247.4, 45.0)
- added R175: 232K 1%, Resistor_SMD:R_0402_1005Metric, F.Cu at (247.4, 47.0)
- added R176: 49.9K 1%, Resistor_SMD:R_0402_1005Metric, F.Cu at (247.4, 49.0)
- added U46: PI6C557-03BLE, lcsc:TSSOP-16_L5.0-W4.4-P0.65-LS6.4-BL, F.Cu at (256.6, 44.3)
- added U50: TP5108E23E-33, lcsc:SOT-23-5_L3.0-W1.7-P0.95-LS2.8-BL, F.Cu at (242.6, 62.4)
- added U51: SY8089AAAC, lcsc:SOT-23-5_L3.0-W1.7-P0.95-LS2.8-BR, F.Cu at (247.0, 62.3)
- added X6: X322525MOB4SI, lcsc:CRYSTAL-SMD_4P-L3.2-W2.5-BL, F.Cu at (259.4, 62.1)
- moved RJ1 4.48 mm to (25.8, 116.8)
Connections:
- CN2 pad 50: unconnected-(CN2-Pad50) -> Net-(CN2-Pad50)
- CN2 pad 52: unconnected-(CN2-Pad52) -> Net-(CN2-Pad52)
- CN2 pad 54: unconnected-(CN2-Pad54) -> Net-(CN2-Pad54)

Commit message: sensors
Parts:
- added C322: 1uF X5R 6.3V, Capacitor_SMD:C_0402_1005Metric, F.Cu at (239.2, 85.1)
- added C323: 100nF X5R 10V, Capacitor_SMD:C_0402_1005Metric, F.Cu at (239.2, 87.1)
- added C324: 1uF X5R 6.3V, Capacitor_SMD:C_0402_1005Metric, F.Cu at (239.2, 89.1)
- added C325: 1uF X5R 6.3V, Capacitor_SMD:C_0402_1005Metric, F.Cu at (239.2, 91.0)
- added C326: 1uF X5R 6.3V, Capacitor_SMD:C_0402_1005Metric, F.Cu at (242.1, 85.1)
- added C327: 100nF X5R 10V, Capacitor_SMD:C_0402_1005Metric, F.Cu at (242.1, 87.1)
- added C328: 100nF X5R 10V, Capacitor_SMD:C_0402_1005Metric, F.Cu at (242.1, 89.1)
- added C329: 100nF X5R 10V, Capacitor_SMD:C_0402_1005Metric, F.Cu at (242.1, 91.0)
- added C330: 100nF X5R 10V, Capacitor_SMD:C_0402_1005Metric, F.Cu at (244.9, 85.1)
- added C331: 100nF X5R 10V, Capacitor_SMD:C_0402_1005Metric, F.Cu at (244.9, 87.1)
- added C332: 1uF X5R 6.3V, Capacitor_SMD:C_0402_1005Metric, F.Cu at (244.9, 89.1)
- added C333: 100nF X5R 16V, Capacitor_SMD:C_0402_1005Metric, F.Cu at (244.9, 91.0)
- added R177: 10K 5%, Resistor_SMD:R_0402_1005Metric, F.Cu at (248.5, 93.0)
- added R178: 15R 5%, Resistor_SMD:R_0402_1005Metric, F.Cu at (248.5, 95.0)
- added R179: 10K 5%, Resistor_SMD:R_0402_1005Metric, F.Cu at (248.5, 97.0)
- added U52: MXC6655XA, lcsc:LGA-12_L2.0-W2.0-P0.50-TL_BOSCH_BMA490L, F.Cu at (248.3, 90.2)
- added U53: AK09918C, lcsc:WLCSP-4_L0.8-W0.8-R2-C2-P0.40-BL-1, F.Cu at (244.4, 98.1)
- added U54: SC7A20TR_C5126709, lcsc:LGA-12_L2.0-W2.0-P0.50-BL, F.Cu at (239.6, 97.8)
- added U55: ICM-20600, lcsc:LGA-14_L3.0-W2.5-P0.50-BL, F.Cu at (245.0, 94.3)
- added U56: STK3311-X_C966926, lcsc:LGA-8_L4.0-W2.4-P0.97-BR, F.Cu at (240.4, 93.9)
- added U57: HAL248TDSO, lcsc:SOT-23-3_L2.9-W1.6-P1.90-LS2.8-BR-CW, F.Cu at (248.7, 86.2)

Commit message: finished schematic!
Parts:
- added C334: 10uF X5R 10V, Capacitor_SMD:C_0603_1608Metric, F.Cu at (261.1, 131.8)
- added C335: 100nF X5R 10V, Capacitor_SMD:C_0402_1005Metric, F.Cu at (257.6, 137.5)
- added C336: 10uF X5R 10V, Capacitor_SMD:C_0603_1608Metric, F.Cu at (261.1, 134.3)
- added C337: 100nF X5R 10V, Capacitor_SMD:C_0201_0603Metric, F.Cu at (260.4, 146.7)
- added C338: 100nF X5R 10V, Capacitor_SMD:C_0201_0603Metric, F.Cu at (260.4, 148.4)
- added C339: 100nF X5R 10V, Capacitor_SMD:C_0402_1005Metric, F.Cu at (268.0, 142.8)
- added C340: 100nF X5R 10V, Capacitor_SMD:C_0201_0603Metric, F.Cu at (265.4, 142.7)
- added C341: 4.7uF X5R 6.3V, Capacitor_SMD:C_0402_1005Metric, F.Cu at (268.0, 144.8)
- added C342: 100nF X5R 10V, Capacitor_SMD:C_0201_0603Metric, F.Cu at (265.4, 144.4)
- added C343: 4.7uF X5R 6.3V, Capacitor_SMD:C_0402_1005Metric, F.Cu at (268.0, 146.7)
- added C344: 100nF X5R 10V, Capacitor_SMD:C_0201_0603Metric, F.Cu at (265.4, 146.2)
- added C345: 100nF X5R 10V, Capacitor_SMD:C_0201_0603Metric, F.Cu at (265.4, 147.9)
- added C346: 100nF X5R 10V, Capacitor_SMD:C_0201_0603Metric, F.Cu at (265.4, 149.7)
- added C347: 4.7uF X5R 6.3V, Capacitor_SMD:C_0402_1005Metric, F.Cu at (268.0, 153.5)
- added C348: 100nF X5R 10V, Capacitor_SMD:C_0201_0603Metric, F.Cu at (265.4, 153.4)
- added C349: 100nF X5R 10V, Capacitor_SMD:C_0201_0603Metric, F.Cu at (265.4, 155.2)
- added C350: 4.7uF X5R 6.3V, Capacitor_SMD:C_0402_1005Metric, F.Cu at (268.0, 155.5)
- added C351: 100nF X5R 10V, Capacitor_SMD:C_0201_0603Metric, F.Cu at (228.2, 150.5)
- added C352: 100nF X5R 10V, Capacitor_SMD:C_0201_0603Metric, F.Cu at (228.2, 146.8)
- added C353: 1nF X5R 10V, Capacitor_SMD:C_0402_1005Metric, F.Cu at (221.0, 141.4)
- added C354: 1nF X5R 10V, Capacitor_SMD:C_0402_1005Metric, F.Cu at (221.0, 143.3)
- added C355: 1nF X5R 10V, Capacitor_SMD:C_0402_1005Metric, F.Cu at (221.0, 145.3)
- added C356: 1nF X5R 10V, Capacitor_SMD:C_0402_1005Metric, F.Cu at (221.0, 147.3)
- added C357: 1nF X5R 10V, Capacitor_SMD:C_0402_1005Metric, F.Cu at (221.0, 149.2)
- added C358: 100nF X5R 10V, Capacitor_SMD:C_0201_0603Metric, F.Cu at (223.7, 141.2)
- added C359: 100nF X5R 10V, Capacitor_SMD:C_0201_0603Metric, F.Cu at (223.7, 143.0)
- added C360: 100nF X5R 10V, Capacitor_SMD:C_0201_0603Metric, F.Cu at (228.2, 141.2)
- added C361: 100nF X5R 10V, Capacitor_SMD:C_0201_0603Metric, F.Cu at (228.2, 143.0)
- added C362: 100nF X5R 10V, Capacitor_SMD:C_0201_0603Metric, F.Cu at (134.5, 11.9)
- added C363: 1uF X5R 6.3V, Capacitor_SMD:C_0402_1005Metric, F.Cu at (131.9, 12.0)
- added C364: 100nF X5R 10V, Capacitor_SMD:C_0201_0603Metric, F.Cu at (123.7, 9.54)
- added C365: 100nF X5R 10V, Capacitor_SMD:C_0201_0603Metric, F.Cu at (192.7, 137.2)
- added C366: 4.7uF X5R 6.3V, Capacitor_SMD:C_0402_1005Metric, F.Cu at (190.0, 137.4)
- added C367: 100nF X5R 10V, Capacitor_SMD:C_0201_0603Metric, F.Cu at (192.7, 139.0)
- added C368: 4.7uF X5R 6.3V, Capacitor_SMD:C_0402_1005Metric, F.Cu at (190.0, 139.3)
- added C369: 100nF X5R 10V, Capacitor_SMD:C_0201_0603Metric, F.Cu at (189.8, 143.2)
- added C370: 100nF X5R 10V, Capacitor_SMD:C_0201_0603Metric, F.Cu at (189.8, 144.9)
- added C371: 100nF X5R 10V, Capacitor_SMD:C_0201_0603Metric, F.Cu at (192.7, 131.3)
- added C372: 100nF X5R 10V, Capacitor_SMD:C_0201_0603Metric, F.Cu at (192.7, 121.3)
- added J4: Conn_01x04, Connector_PinHeader_2.54mm:PinHeader_1x04_P2.54mm_Vertical, F.Cu at (247.7, 140.8)
- added L12: L_Iron_Coupled_Small, lcsc:FILTER-SMD_4P-L2.0-W1.2-BL_DLW21H, F.Cu at (123.9, 6.87)
- added Q9: WPM2015-3/TR_C7472861, lcsc:SOT-23-3_L2.9-W1.3-P1.90-LS2.4-BR, F.Cu at (261.2, 137.7)
- added R180: 100R 5%, Resistor_SMD:R_0402_1005Metric, F.Cu at (246.9, 131.6)
- added R181: 100R 5%, Resistor_SMD:R_0402_1005Metric, F.Cu at (246.9, 133.6)
- added R182: 120R 5%, Resistor_SMD:R_0402_1005Metric, F.Cu at (246.9, 135.5)
- added R183: 100R 5%, Resistor_SMD:R_0402_1005Metric, F.Cu at (246.9, 137.5)
- added R184: 100R 5%, Resistor_SMD:R_0402_1005Metric, F.Cu at (249.8, 131.6)
- added R185: 100R 5%, Resistor_SMD:R_0402_1005Metric, F.Cu at (249.8, 133.6)
- added R186: 10K 1%, Resistor_SMD:R_0402_1005Metric, F.Cu at (249.8, 135.5)
- added R187: 10K 1%, Resistor_SMD:R_0402_1005Metric, F.Cu at (249.8, 137.5)
- added R188: 10K 1%, Resistor_SMD:R_0402_1005Metric, F.Cu at (252.7, 131.6)
- added R189: 10K 1%, Resistor_SMD:R_0402_1005Metric, F.Cu at (252.7, 133.6)
- added R190: 10K 5%, Resistor_SMD:R_0402_1005Metric, F.Cu at (257.6, 131.6)
- added R191: 100K 5%, Resistor_SMD:R_0402_1005Metric, F.Cu at (257.6, 133.6)
- added R192: 100K 5%, Resistor_SMD:R_0402_1005Metric, F.Cu at (257.6, 135.5)
- added R193: 2.2K 5%, Resistor_SMD:R_0402_1005Metric, F.Cu at (252.7, 135.5)
- added R194: 2.2K 5%, Resistor_SMD:R_0402_1005Metric, F.Cu at (252.7, 137.5)
- added R195: 22R 5%, Resistor_SMD:R_0402_1005Metric, F.Cu at (260.7, 142.8)
- added R196: 22R 5%, Resistor_SMD:R_0402_1005Metric, F.Cu at (260.7, 144.8)
- added R197: 200R 1%, Resistor_SMD:R_0201_0603Metric, F.Cu at (265.4, 156.9)
- added R198: 10K 5%, Resistor_SMD:R_0402_1005Metric, F.Cu at (218.0, 147.5)
- added R199: 10K 5%, Resistor_SMD:R_0402_1005Metric, F.Cu at (218.0, 149.5)
- added R200: 2.2K 5%, Resistor_SMD:R_0402_1005Metric, F.Cu at (128.8, 6.07)
- added R201: 2.2K 5%, Resistor_SMD:R_0402_1005Metric, F.Cu at (128.8, 8.06)
- added R202: 22R 5%, Resistor_SMD:R_0402_1005Metric, F.Cu at (128.8, 10.1)
- added R203: 22R 5%, Resistor_SMD:R_0402_1005Metric, F.Cu at (131.8, 6.07)
- added R204: 22R 5%, Resistor_SMD:R_0402_1005Metric, F.Cu at (131.8, 8.06)
- added R205: 22R 5%, Resistor_SMD:R_0402_1005Metric, F.Cu at (131.8, 10.1)
- added R206: 22R 5%, Resistor_SMD:R_0402_1005Metric, F.Cu at (134.7, 6.07)
- added R207: 22R 5%, Resistor_SMD:R_0402_1005Metric, F.Cu at (134.7, 8.06)
- added R208: 0R 5%, Resistor_SMD:R_0402_1005Metric, F.Cu at (134.7, 10.1)
- added R209: 2.2R 5%, Resistor_SMD:R_0402_1005Metric, F.Cu at (121.0, 6.07)
- added R210: 2.2R 5%, Resistor_SMD:R_0402_1005Metric, F.Cu at (121.0, 8.06)
- added R211: 2.2R 5%, Resistor_SMD:R_0402_1005Metric, F.Cu at (121.0, 10.1)
- added R212: 2.2R 5%, Resistor_SMD:R_0402_1005Metric, F.Cu at (121.0, 12.0)
- added R213: 2.2R 5%, Resistor_SMD:R_0402_1005Metric, F.Cu at (121.0, 14.0)
- added R214: 2.2R 5%, Resistor_SMD:R_0402_1005Metric, F.Cu at (121.0, 16.0)
- added R215: 2.2R 5%, Resistor_SMD:R_0402_1005Metric, F.Cu at (121.0, 18.0)
- added R216: 2.2R 5%, Resistor_SMD:R_0402_1005Metric, F.Cu at (121.0, 20.0)
- added R217: 1.62K 1%, Resistor_SMD:R_0201_0603Metric, F.Cu at (123.7, 11.3)
- added R218: 2.2K 5%, Resistor_SMD:R_0402_1005Metric, F.Cu at (190.0, 131.4)
- added R219: 2.2K 5%, Resistor_SMD:R_0402_1005Metric, F.Cu at (190.0, 133.4)
- added R220: 22R 5%, Resistor_SMD:R_0402_1005Metric, F.Cu at (190.0, 121.4)
- added R221: 22R 5%, Resistor_SMD:R_0402_1005Metric, F.Cu at (190.0, 123.4)
- added R223: 22R 5%, Resistor_SMD:R_0402_1005Metric, F.Cu at (190.0, 125.4)
- added R224: 22R 5%, Resistor_SMD:R_0402_1005Metric, F.Cu at (190.0, 127.4)
- added SW1: TS24CA, lcsc:SW-SMD_2P-TS24CA, F.Cu at (242.2, 133.6)
- added SW2: TS24CA, lcsc:SW-SMD_2P-TS24CA, F.Cu at (242.2, 138.7)
- added SW3: TS24CA, lcsc:SW-SMD_2P-TS24CA, F.Cu at (242.2, 143.8)
- added TP10: TestPoint, TestPoint:TestPoint_Pad_D1.0mm, F.Cu at (218.1, 141.9)
- added TP11: TestPoint, TestPoint:TestPoint_Pad_D1.0mm, F.Cu at (218.1, 144.9)
- added TP12: TestPoint, TestPoint:TestPoint_Pad_D1.0mm, F.Cu at (128.9, 12.6)
- added TP5: TestPoint, TestPoint:TestPoint_Pad_D1.0mm, F.Cu at (257.7, 143.3)
- added TP6: TestPoint, TestPoint:TestPoint_Pad_D1.0mm, F.Cu at (257.7, 146.4)
- added TP7: TestPoint, TestPoint:TestPoint_Pad_D1.0mm, F.Cu at (257.7, 149.4)
- added TP8: TestPoint, TestPoint:TestPoint_Pad_D1.0mm, F.Cu at (257.7, 152.5)
- added TP9: TestPoint, TestPoint:TestPoint_Pad_D1.0mm, F.Cu at (257.7, 155.5)
- added U58: ESD5451N_C5261080, lcsc:DFN1006-2L-BI, F.Cu at (251.4, 139.5)
- added U59: ESD5451N_C5261080, lcsc:DFN1006-2L-BI, F.Cu at (251.4, 141.4)
- added U60: ESD5451N_C5261080, lcsc:DFN1006-2L-BI, F.Cu at (251.4, 143.3)
- added U61: ESD5451N_C5261080, lcsc:DFN1006-2L-BI, F.Cu at (251.4, 145.2)
- added U62: ESD5451N_C5261080, lcsc:DFN1006-2L-BI, F.Cu at (251.4, 147.1)
- C198: value 1uF X5R 10V -> 100nF X5R 10V
- C199: value 10pF C0G 50V -> 100nF X5R 10V
- C2: value 10pF C0G -> 10pF C0G 50V
- CN2: value 35RAPC4BH3 -> 1-2199230-5; footprint lcsc:AUDIO-TH_35RAPC4BH3 -> lcsc:PCIE-SMD_75P-P0.50_1-2199230-5
- R1: value 22R -> 22R 5%
- R129: value 100R 5% -> 1K 5%
- R139: value 2.2K 5% -> 100K 5%
- R2: value 1M -> 1M 5%
- U46: value ESD5451N_C5261080 -> PI6C557-03BLE; footprint lcsc:DFN1006-2L-BI -> lcsc:TSSOP-16_L5.0-W4.4-P0.65-LS6.4-BL
- moved U2 10.4 mm to (157.0, 77.5)
- moved U1 0.80 mm to (167.8, 94.3)
Connections:
- net GMAC0_INT/PMEB_GPIO3_C0 renamed GMAC1_INT/PMEB_GPIO3_A7
- net GMAC0_RSTn_GPIO3_B0 renamed GMAC1_RSTn_GPIO3_B0
- C198 pad 1: Net-(C198-Pad1) -> HP_DET_L_GPIO3_C2
- C199 pad 1: MIC1_INP -> VDD_CPU
- C42 pad 2: GND -> Net-(Q3-G)
- CN2 pad 1: unconnected-(CN2-Pad1) -> GND
- CN2 pad 2: unconnected-(CN2-Pad2) -> VCC3V3_PCIE30
- CN2 pad 3: unconnected-(CN2-Pad3) -> GND
- CN2 pad 4: unconnected-(CN2-Pad4) -> VCC3V3_PCIE30
- D12 pad 10: /HDMI/HDMI_TX2P_PORT -> HDMI_TX2P_PORT
- D12 pad 6: /HDMI/HDMI_TX1N_PORT -> HDMI_TX1N_PORT
- D12 pad 7: /HDMI/HDMI_TX1P_PORT -> HDMI_TX1P_PORT
- D12 pad 9: /HDMI/HDMI_TX2N_PORT -> HDMI_TX2N_PORT
- D13 pad 10: /HDMI/HDMI_TXCLKN_PORT -> HDMI_TXCLKN_PORT
- D13 pad 6: /HDMI/HDMI_TX0P_PORT -> HDMI_TX0P_PORT
- D13 pad 7: /HDMI/HDMI_TX0N_PORT -> HDMI_TX0N_PORT
- D13 pad 9: /HDMI/HDMI_TXCLKP_PORT -> HDMI_TXCLKP_PORT
- FPC1 pad 27: LCD_RST_L_GPIO3_C7 -> LCD_RST_L_GPIO2_D6
- Q6 pad 2: /HDMI/HDMITX_SCL -> HDMITX_SCL
- Q7 pad 2: /HDMI/HDMITX_SDA -> HDMITX_SDA
- Q8 pad 2: /HDMI/HDMITX_CEC_M0 -> HDMITX_CEC_M0
- R1 pad 1: Net-(C1-Pad1) -> /Peripherals/XOUT24M
- R1 pad 2: /Peripherals/XOUT24M -> Net-(C1-Pad1)
- R10 pad 1: /Power/USB3_OTG0_SSRXN -> USB3_OTG0_SSRXN
- R100 pad 2: GMAC0_MCLKINOUT -> GMAC1_MCLKINOUT_M1
- R101 pad 1: GMAC0_MCLKINOUT -> GMAC1_MCLKINOUT_M1
- R105 pad 1: GMAC0_MDIO -> GMAC1_MDIO_M1
- R106 pad 1: GMAC0_RXD0 -> GMAC1_RXD0_M1
- R107 pad 1: GMAC0_RXD1 -> GMAC1_RXD1_M1
- R108 pad 1: GMAC0_RXD2 -> GMAC1_RXD2_M1
- R109 pad 1: GMAC0_RXD3 -> GMAC1_RXD3_M1
- R11 pad 1: /Power/USB3_OTG0_SSRXP -> USB3_OTG0_SSRXP
- R110 pad 1: GMAC0_RXCLK -> GMAC1_RXCLK_M1
- R111 pad 1: GMAC0_RXDV_CRS -> GMAC1_RXDV_CRS_M1
- R129 pad 1: Net-(C198-Pad1) -> Net-(CN1-Pad3)
- R129 pad 2: VCCIO_ACODEC -> HP_DET_L_GPIO3_C2
- R139 pad 1: MIC1_INP -> VCC_1V8
- R139 pad 2: Net-(C198-Pad1) -> HP_DET_L_GPIO3_C2
- R2 pad 1: /Peripherals/XIN24M -> /Peripherals/XOUT24M
- R2 pad 2: /Peripherals/XOUT24M -> /Peripherals/XIN24M
- R64 pad 2: USB3_OTG0_DP -> USB3_HOST1_DP
- R65 pad 2: USB3_OTG0_DM -> USB3_HOST1_DM
- R81 pad 2: DVP_PWREN0_H_GPIO0_D3 -> MIPI_CAM0_RST_L_GPIO3_C6
- R83 pad 2: /HDMI/HDMITX_SCL -> HDMITX_SCL
- R84 pad 2: /HDMI/HDMITX_SDA -> HDMITX_SDA
- R86 pad 2: /HDMI/HDMITX_CEC_M0 -> HDMITX_CEC_M0
- R87 pad 1: /HDMI/HDMI_TX_HPDIN -> HDMI_TX_HPDIN
- R89 pad 2: /Display/LCD0_BL_PWM4 -> LCD0_BL_PWM4
- U1 pad A19: unconnected-(U1G-GPIO1_A2_D-PadA19) -> Net-(U1G-GPIO1_A2_D)
- U1 pad A20: unconnected-(U1G-GPIO1_A5_D-PadA20) -> Net-(U1G-GPIO1_A5_D)
- U1 pad A23: unconnected-(U1H-GPIO1_C5_D-PadA23) -> Net-(U1H-GPIO1_C5_D)
- U1 pad A24: unconnected-(U1H-GPIO1_B4_U-PadA24) -> eMMC_D0
- U1 pad A25: unconnected-(U1H-GPIO1_C0_U-PadA25) -> eMMC_D4
- U1 pad A26: unconnected-(U1H-GPIO1_C6_D-PadA26) -> eMMC_DATA_STROBE
- U1 pad AA11: unconnected-(U1M-GPIO4_C3_D-PadAA11) -> PCIE30X2_WAKEn_M2
- U1 pad AA18: unconnected-(U1P-HDMI_TX_REXT-PadAA18) -> Net-(U1P-HDMI_TX_REXT)
- U1 pad AA2: unconnected-(U1L-GPIO4_A1_D-PadAA2) -> GMAC1_RXD2_M1
- U1 pad AA22: unconnected-(U1F-GPIO0_A3_U-PadAA22) -> PMIC_INT_L
- U1 pad AA25: unconnected-(U1V-PCIE30_REFCLKN_IN-PadAA25) -> PCIE30_REFCLKN_IN
- U1 pad AA27: unconnected-(U1V-PCIE30_TX0N-PadAA27) -> PCIE30_TX0N
- U1 pad AA28: unconnected-(U1V-PCIE30_TX0P-PadAA28) -> PCIE30_TX0P
- U1 pad AA3: unconnected-(U1L-GPIO4_A0_D-PadAA3) -> Net-(U1L-GPIO4_A0_D)
- U1 pad AA6: unconnected-(U1L-GPIO3_C7_D-PadAA6) -> MIPI_CAM0_PDN_L_GPIO3_C7
- U1 pad AA7: unconnected-(U1K-GPIO3_C2_D-PadAA7) -> HP_DET_L_GPIO3_C2
- U1 pad AB18: unconnected-(U1P-HDMI_TX_HPDIN-PadAB18) -> HDMI_TX_HPDIN
- U1 pad AB21: unconnected-(U1F-GPIO0_B2_U-PadAB21) -> I2C0_SDA_PMIC
- U1 pad AB27: unconnected-(U1V-PCIE30_TX1N-PadAB27) -> PCIE30_TX1N
- U1 pad AB28: unconnected-(U1V-PCIE30_TX1P-PadAB28) -> PCIE30_TX1P
- U1 pad AB9: unconnected-(U1M-GPIO4_D2_D-PadAB9) -> TYPEC_SW_SEL_GPIO4_D2
- U1 pad AC20: unconnected-(U1F-GPIO0_D0_U-PadAC20) -> UART2_RX_M0_DEBUG
- U1 pad AC21: unconnected-(U1F-GPIO0_C5_D-PadAC21) -> USBCC_INT_L_GPIO0_C5
- U1 pad AC27: unconnected-(U1V-PCIE30_RX0N-PadAC27) -> PCIE30_RX0N
- U1 pad AC28: unconnected-(U1V-PCIE30_RX0P-PadAC28) -> PCIE30_RX0P
- U1 pad AC4: unconnected-(U1K-GPIO3_C3_D-PadAC4) -> BQ_OTG_EN_H_GPIO3_C3
- U1 pad AC5: unconnected-(U1L-GPIO3_C6_D-PadAC5) -> MIPI_CAM0_RST_L_GPIO3_C6
- U1 pad AC7: unconnected-(U1K-GPIO2_D3_D-PadAC7) -> ALPS_INT_L_GPIO2_D3
- U1 pad AC8: unconnected-(U1K-GPIO2_D2_D-PadAC8) -> GSENSOR_INT_L_GPIO2_D2
- U1 pad AD1: unconnected-(U1K-GPIO3_C1_D-PadAD1) -> PCIE20_PERSTn_M1
- U1 pad AD11: unconnected-(U1O-MIPI_CSI_RX_D2N-PadAD11) -> MIPI_CSI_RX_D2N
- U1 pad AD20: unconnected-(U1F-GPIO0_C6_D-PadAD20) -> HALL_INT_L_GPIO0_C6
- U1 pad AD21: unconnected-(U1F-GPIO0_C4_D-PadAD21) -> WIFI_WAKE_HOST_H_GPIO0_C4
- U1 pad AD22: unconnected-(U1F-GPIO0_C0_D-PadAD22) -> WIFI_REG_ON_H_GPIO0_C0
- U1 pad AD23: unconnected-(U1F-GPIO0_B0_U-PadAD23) -> HOST_WAKE_BT_H_GPIO0_B0
- U1 pad AD25: 4G_PWREN_H_GPIO0_D5 -> unconnected-(U1F-GPIO0_D5_D-PadAD25)
- U1 pad AD27: unconnected-(U1V-PCIE30_RX1N-PadAD27) -> PCIE30_RX1N
- U1 pad AD28: unconnected-(U1V-PCIE30_RX1P-PadAD28) -> PCIE30_RX1P
- U1 pad AD6: unconnected-(U1K-GPIO2_D6_D-PadAD6) -> LCD_RST_L_GPIO2_D6
- U1 pad AD7: unconnected-(U1K-GPIO2_D1_D-PadAD7) -> PCIE20_WAKEn_M1
- U1 pad AD9: unconnected-(U1O-MIPI_CSI_RX_D3P-PadAD9) -> MIPI_CSI_RX_D3P
- U1 pad AE1: unconnected-(U1K-GPIO3_B4_D-PadAE1) -> I2C5_SDA_M0
- U1 pad AE11: unconnected-(U1O-MIPI_CSI_RX_D2P-PadAE11) -> MIPI_CSI_RX_D2P
- U1 pad AE23: unconnected-(U1F-GPIO0_C3_D-PadAE23) -> LCD0_BL_PWM4
- U1 pad AE24: unconnected-(U1F-GPIO0_A6_D-PadAE24) -> USB_HOST_PWREN_H_GPIO0_A6
- U1 pad AE9: unconnected-(U1O-MIPI_CSI_RX_D3N-PadAE9) -> MIPI_CSI_RX_D3N
- U1 pad AF1: unconnected-(U1K-GPIO3_B3_D-PadAF1) -> I2C5_SCL_M0
- U1 pad AF23: unconnected-(U1F-GPIO0_C1_D-PadAF23) -> BT_REG_ON_H_GPIO0_C1
- U1 pad AF24: unconnected-(U1F-GPIO0_B1_U-PadAF24) -> I2C0_SCL_PMIC
- U1 pad AF25: unconnected-(U1F-GPIO0_A5_D-PadAF25) -> SDMMC0_PWREN_L
- U1 pad AF5: unconnected-(U1K-GPIO2_D4_D-PadAF5) -> GYRO_INT_L_GPIO2_D4
- U1 pad AF6: unconnected-(U1K-GPIO2_D5_D-PadAF6) -> LCD_EN_H_GPIO2_D5
- U1 pad AF8: unconnected-(U1M-GPIO4_C2_D-PadAF8) -> PCIE30X2_CLKREQn_M2
- U1 pad AG10: unconnected-(U1O-MIPI_CSI_RX_CLK0P-PadAG10) -> MIPI_CSI_RX_CLK0P
- U1 pad AG11: unconnected-(U1O-MIPI_CSI_RX_D1P-PadAG11) -> MIPI_CSI_RX_D1P
- U1 pad AG12: unconnected-(U1O-MIPI_CSI_RX_D0P-PadAG12) -> MIPI_CSI_RX_D0P
- U1 pad AG13: unconnected-(U1Q-MIPI_DSI_TX0_D3N/LVDS_TX0_D3N-PadAG13) -> MIPI_DSI_TX0_D3N
- U1 pad AG14: unconnected-(U1Q-MIPI_DSI_TX0_D2N/LVDS_TX0_D2N-PadAG14) -> MIPI_DSI_TX0_D2N
- U1 pad AG15: unconnected-(U1Q-MIPI_DSI_TX0_CLKN/LVDS_TX0_CLKN-PadAG15) -> MIPI_DSI_TX0_CLKN
- U1 pad AG16: unconnected-(U1Q-MIPI_DSI_TX0_D1N/LVDS_TX0_D1N-PadAG16) -> MIPI_DSI_TX0_D1N
- U1 pad AG17: unconnected-(U1Q-MIPI_DSI_TX0_D0N/LVDS_TX0_D0N-PadAG17) -> MIPI_DSI_TX0_D0N
- U1 pad AG19: unconnected-(U1P-HDMI_TX_CLKN-PadAG19) -> Net-(U1P-HDMI_TX_CLKN)
- U1 pad AG20: unconnected-(U1P-HDMI_TX_D0P-PadAG20) -> Net-(U1P-HDMI_TX_D0P)
- U1 pad AG21: unconnected-(U1P-HDMI_TX_D1P-PadAG21) -> Net-(U1P-HDMI_TX_D1P)
- U1 pad AG22: unconnected-(U1P-HDMI_TX_D2P-PadAG22) -> Net-(U1P-HDMI_TX_D2P)
- U1 pad AG23: unconnected-(U1F-GPIO0_C2_D-PadAG23) -> CHG_INT_L_GPIO0_C2
- U1 pad AG25: unconnected-(U1F-GPIO0_A7_U-PadAG25) -> FLASH_VOL_SEL
- U1 pad AG26: unconnected-(U1F-GPIO0_A1_Z-PadAG26) -> TSADC_SHUT_M0
- U1 pad AG27: unconnected-(U1F-GPIO0_A0_D-PadAG27) -> WIFI_PWREN_GPIO0_A0
- U1 pad AG28: unconnected-(U1F-GPIO0_A2_D-PadAG28) -> PMIC_SLEEP_H
- U1 pad AG6: unconnected-(U1K-GPIO2_D0_D-PadAG6) -> PCIE20_CLKREQn_M1
- U1 pad AG7: unconnected-(U1M-GPIO4_D0_U-PadAG7) -> HDMITX_SDA
- U1 pad AG8: unconnected-(U1M-GPIO4_C7_U-PadAG8) -> HDMITX_SCL
- U1 pad AG9: unconnected-(U1O-MIPI_CSI_RX_CLK1P-PadAG9) -> MIPI_CSI_RX_CLK1P
- U1 pad AH10: unconnected-(U1O-MIPI_CSI_RX_CLK0N-PadAH10) -> MIPI_CSI_RX_CLK0N
- U1 pad AH11: unconnected-(U1O-MIPI_CSI_RX_D1N-PadAH11) -> MIPI_CSI_RX_D1N
- U1 pad AH12: unconnected-(U1O-MIPI_CSI_RX_D0N-PadAH12) -> MIPI_CSI_RX_D0N
- U1 pad AH13: unconnected-(U1Q-MIPI_DSI_TX0_D3P/LVDS_TX0_D3P-PadAH13) -> MIPI_DSI_TX0_D3P
- U1 pad AH14: unconnected-(U1Q-MIPI_DSI_TX0_D2P/LVDS_TX0_D2P-PadAH14) -> MIPI_DSI_TX0_D2P
- U1 pad AH15: unconnected-(U1Q-MIPI_DSI_TX0_CLKP/LVDS_TX0_CLKP-PadAH15) -> MIPI_DSI_TX0_CLKP
- U1 pad AH16: unconnected-(U1Q-MIPI_DSI_TX0_D1P/LVDS_TX0_D1P-PadAH16) -> MIPI_DSI_TX0_D1P
- U1 pad AH17: unconnected-(U1Q-MIPI_DSI_TX0_D0P/LVDS_TX0_D0P-PadAH17) -> MIPI_DSI_TX0_D0P
- U1 pad AH19: unconnected-(U1P-HDMI_TX_CLKP-PadAH19) -> Net-(U1P-HDMI_TX_CLKP)
- U1 pad AH20: unconnected-(U1P-HDMI_TX_D0N-PadAH20) -> Net-(U1P-HDMI_TX_D0N)
- U1 pad AH21: unconnected-(U1P-HDMI_TX_D1N-PadAH21) -> Net-(U1P-HDMI_TX_D1N)
- U1 pad AH22: unconnected-(U1P-HDMI_TX_D2N-PadAH22) -> Net-(U1P-HDMI_TX_D2N)
- U1 pad AH24: unconnected-(U1F-GPIO0_D1_U-PadAH24) -> UART2_TX_M0_DEBUG
- U1 pad AH25: unconnected-(U1F-GPIO0_C7_D-PadAH25) -> LCD0_PWREN_H_GPIO0_C7
- U1 pad AH26: unconnected-(U1F-GPIO0_B7_D-PadAH26) -> BT_WAKE_HOST_H_GPIO0_B7
- U1 pad AH6: unconnected-(U1M-GPIO4_D1_U-PadAH6) -> HDMITX_CEC_M0
- U1 pad AH7: unconnected-(U1M-GPIO4_C4_D-PadAH7) -> PCIE30X2_PERSTn_M2
- U1 pad AH9: unconnected-(U1O-MIPI_CSI_RX_CLK1N-PadAH9) -> MIPI_CSI_RX_CLK1N
- U1 pad B19: unconnected-(U1G-GPIO1_A3_D-PadB19) -> Net-(U1G-GPIO1_A3_D)
- U1 pad B20: unconnected-(U1G-GPIO1_A7_D-PadB20) -> I2S1_SDO0_M0_PMIC
- U1 pad B21: unconnected-(U1G-GPIO1_B3_D-PadB21) -> I2S1_SDI0_M0/PDM_SDI0_M0_PMIC
- U1 pad B22: unconnected-(U1H-GPIO1_C4_U-PadB22) -> eMMC_CMD
- U1 pad B24: unconnected-(U1H-GPIO1_B6_U-PadB24) -> eMMC_D2
- U1 pad B25: unconnected-(U1H-GPIO1_C3_U-PadB25) -> eMMC_D7
- U1 pad B27: unconnected-(U1N-SARADC_VIN0-PadB27) -> SARADC_VIN0_KEY/RECOVERY
- U1 pad C20: unconnected-(U1G-GPIO1_A6_D-PadC20) -> Net-(U1G-GPIO1_A6_D)
- U1 pad C21: unconnected-(U1H-GPIO1_B5_U-PadC21) -> eMMC_D1
- U1 pad C26: unconnected-(U1N-SARADC_VIN1-PadC26) -> SARADC_VIN1_HW_ID
- U1 pad D21: unconnected-(U1H-GPIO1_B7_U-PadD21) -> eMMC_D3
- U1 pad D24: unconnected-(U1N-SARADC_VIN2-PadD24) -> SARADC_VIN2_HP_HOOK
- U1 pad E21: unconnected-(U1H-GPIO1_C1_U-PadE21) -> eMMC_D5
- U1 pad E22: unconnected-(U1H-GPIO1_C2_U-PadE22) -> eMMC_D6
- U1 pad E23: unconnected-(U1N-SARADC_VIN3-PadE23) -> SARADC_VIN3_BOM_ID
- U1 pad F20: unconnected-(U1H-GPIO1_C7_D-PadF20) -> eMMC_RSTn
- U1 pad F25: unconnected-(U1J-GPIO2_C2_D-PadF25) -> SOC_PCM_CLK
- U1 pad F26: unconnected-(U1J-GPIO2_C5_D-PadF26) -> SOC_PCM_IN
- U1 pad F27: unconnected-(U1J-GPIO2_B6_U-PadF27) -> UART1_CTSn_M0
- U1 pad F28: unconnected-(U1J-GPIO2_B3_U-PadF28) -> UART1_RX_M0
- U1 pad G21: unconnected-(U1N-SARADC_VIN4-PadG21) -> BATT_TC_L
- U1 pad G27: unconnected-(U1J-GPIO2_B4_U-PadG27) -> UART1_TX_M0
- U1 pad G28: unconnected-(U1J-GPIO2_B5_U-PadG28) -> UART1_RTSn_M0
- U1 pad H17: unconnected-(U1G-VCCIO1-PadH17) -> VCCIO_ACODEC
- U1 pad H18: unconnected-(U1H-VCCIO2-PadH18) -> VCCIO_FLASH
- U1 pad H20: unconnected-(U1N-OTP_VCC18-PadH20) -> VCC_1V8
- U1 pad H22: unconnected-(U1N-SARADC_AVDD_1V8-PadH22) -> VCCA_1V8
- U1 pad H23: unconnected-(U1J-GPIO2_C4_D-PadH23) -> SOC_PCM_OUT
- U1 pad H24: unconnected-(U1J-GPIO2_C3_D-PadH24) -> SOC_PCM_SYNC
- U1 pad H26: unconnected-(U1I-GPIO1_D7_U-PadH26) -> SDMMC0_D2/ARMJTAG_TCK
- U1 pad H27: unconnected-(U1I-GPIO2_A1_U-PadH27) -> SDMMC0_CMD
- U1 pad H28: unconnected-(U1I-GPIO2_A2_D-PadH28) -> Net-(U1I-GPIO2_A2_D)
- U1 pad J21: unconnected-(U1J-VCCIO4-PadJ21) -> VCCIO_WL
- U1 pad J23: unconnected-(U1I-GPIO2_A0_U-PadJ23) -> SDMMC0_D3/ARMJTAG_TMS
- U1 pad J24: unconnected-(U1I-GPIO1_D6_U-PadJ24) -> SDMMC0_D1
- U1 pad J25: unconnected-(U1I-GPIO1_D5_U-PadJ25) -> SDMMC0_D0
- U1 pad L22: unconnected-(U1I-VCCIO3-PadL22) -> VCCIO_SD
- U1 pad M23: unconnected-(U1T-USB3_AVDD_3V3-PadM23) -> VCC_3V3
- U1 pad M24: unconnected-(U1T-USB3_OTG0_VBUSDET-PadM24) -> USB3_OTG0_VBUSDET
- U1 pad P22: unconnected-(U1T-USB3_AVDD_0V9-PadP22) -> USB_AVDD_0V9
- U1 pad P23: unconnected-(U1T-USB3_AVDD_1V8-PadP23) -> USB_AVDD_1V8
- U1 pad P24: unconnected-(U1T-USB3_HOST1_DP-PadP24) -> USB3_HOST1_DP
- U1 pad P25: unconnected-(U1T-USB3_HOST1_DM-PadP25) -> USB3_HOST1_DM
- U1 pad P27: unconnected-(U1T-USB3_OTG0_DP-PadP27) -> USB3_OTG0_DP
- U1 pad P28: unconnected-(U1T-USB3_OTG0_DM-PadP28) -> USB3_OTG0_DP
- U1 pad R20: MULTI_PHY_AVDD_0V9 -> VDDA_0V9
- U1 pad R21: MULTI_PHY_AVDD_0V9 -> VDDA_0V9
- U1 pad R22: unconnected-(U1T-MULTI_PHY_AVDD_1V8-PadR22) -> VCCA_1V8
- U1 pad R27: unconnected-(U1T-USB3_OTG0_SSRXN/SATA0_RXN-PadR27) -> USB3_OTG0_SSRXP
- U1 pad R28: unconnected-(U1T-USB3_OTG0_SSRXP/SATA0_RXP-PadR28) -> USB3_OTG0_SSRXN
- U1 pad T27: unconnected-(U1T-USB3_OTG0_SSTXN/SATA0_TXN-PadT27) -> USB3_OTG0_SSTXP
- U1 pad T28: unconnected-(U1T-USB3_OTG0_SSTXP/SATA0_TXP-PadT28) -> USB3_OTG0_SSTXN
- U1 pad U19: unconnected-(U1V-PCIE30_RESREF-PadU19) -> Net-(U1V-PCIE30_RESREF)
- U1 pad U2: unconnected-(U1L-GPIO4_C1_D-PadU2) -> GMAC1_MCLKINOUT_M1
- U1 pad U20: PCIE30_AVDD_0V9 -> VDDA_0V9
- U1 pad U21: PCIE30_AVDD_0V9 -> VDDA_0V9
- U1 pad U22: unconnected-(U1V-PCIE30_AVDD_1V8-PadU22) -> VCCA_1V8
- U1 pad U27: unconnected-(U1T-USB3_HOST1_SSRXN/SATA1_RXN/QSGMII_RXN_M0-PadU27) -> USB3_HOST1_SSRXP
- U1 pad U28: unconnected-(U1T-USB3_HOST1_SSRXP/SATA1_RXP/QSGMII_RXP_M0-PadU28) -> USB3_HOST1_SSRXN
- U1 pad U4: unconnected-(U1L-GPIO4_B7_D-PadU4) -> GMAC1_MDIO_M1
- U1 pad U5: unconnected-(U1L-GPIO4_B6_D-PadU5) -> GMAC1_MDC_M1
- U1 pad V10: VCCIO5 -> VCC_1V8
- U1 pad V11: VCCIO5 -> VCC_1V8
- U1 pad V12: unconnected-(U1M-VCCIO7-PadV12) -> VCC_3V3
- U1 pad V17: HDMI_TX_AVDD_0V9 -> VDDA0V9_IMAGE
- U1 pad V18: HDMI_TX_AVDD_0V9 -> VDDA0V9_IMAGE
- U1 pad V2: unconnected-(U1L-GPIO4_B1_D-PadV2) -> GMAC1_RXDV_CRS_M1
- U1 pad V24: unconnected-(U1T-PCIE20_REFCLKP-PadV24) -> PCIE20_REFCLKP
- U1 pad V25: unconnected-(U1T-PCIE20_REFCLKN-PadV25) -> PCIE20_REFCLKN
- U1 pad V27: unconnected-(U1T-USB3_HOST1_SSTXN/SATA1_TXN/QSGMII_TXN_M0-PadV27) -> USB3_HOST1_SSTXP
- U1 pad V28: unconnected-(U1T-USB3_HOST1_SSTXP/SATA1_TXP/QSGMII_TXP_M0-PadV28) -> USB3_HOST1_SSTXN
- U1 pad V4: unconnected-(U1L-GPIO4_B2_D-PadV4) -> Net-(U1L-GPIO4_B2_D)
- U1 pad V5: unconnected-(U1L-GPIO4_B5_D-PadV5) -> I2C2_SCL_M1
- U1 pad V6: unconnected-(U1L-GPIO4_B4_D-PadV6) -> I2C2_SDA_M1
- U1 pad V7: unconnected-(U1L-GPIO4_B0_D-PadV7) -> GMAC1_RXD1_M1
- U1 pad W1: unconnected-(U1L-GPIO4_A7_D-PadW1) -> GMAC1_RXD0_M1
- U1 pad W14: unconnected-(U1O-MIPI_CSI_RX_AVDD_0V9-PadW14) -> MIPI_AVDD_0V9
- U1 pad W16: unconnected-(U1Q-MIPI_DSI_TX0/LVDS_TX0_AVDD_0V9-PadW16) -> MIPI_AVDD_0V9
- U1 pad W18: unconnected-(U1P-HDMI_TX_AVDD_1V8-PadW18) -> VCCA1V8_IMAGE
- U1 pad W2: unconnected-(U1L-GPIO4_A6_D-PadW2) -> Net-(U1L-GPIO4_A6_D)
- U1 pad W27: unconnected-(U1T-PCIE20_TXP/SATA2_TXP/QSGMII_TXP_M1-PadW27) -> PCIE20_TXP
- U1 pad W28: unconnected-(U1T-PCIE20_TXN/SATA2_TXN/QSGMII_TXN_M1-PadW28) -> PCIE20_TXN
- U1 pad Y1: unconnected-(U1L-GPIO4_A5_D-PadY1) -> Net-(U1L-GPIO4_A5_D)
- U1 pad Y14: unconnected-(U1O-MIPI_CSI_RX_AVDD_1V8-PadY14) -> MIPI_AVDD_1V8
- U1 pad Y17: unconnected-(U1Q-MIPI_DSI_TX0/LVDS_TX0_AVDD_1V8-PadY17) -> MIPI_AVDD_1V8
- U1 pad Y2: unconnected-(U1L-GPIO4_A4_D-PadY2) -> Net-(U1L-GPIO4_A4_D)
- U1 pad Y22: unconnected-(U1F-GPIO0_A4_U-PadY22) -> SDMMC0_DET_L
- U1 pad Y25: unconnected-(U1V-PCIE30_REFCLKP_IN-PadY25) -> PCIE30_REFCLKP_IN
- U1 pad Y27: unconnected-(U1T-PCIE20_RXP/SATA2_RXP/QSGMII_RXP_M1-PadY27) -> PCIE20_RXP
- U1 pad Y28: unconnected-(U1T-PCIE20_RXN/SATA2_RXN/QSGMII_RXN_M1-PadY28) -> PCIE20_RXN
- U1 pad Y3: unconnected-(U1L-GPIO4_A3_D-PadY3) -> GMAC1_RXCLK_M1
- U1 pad Y4: unconnected-(U1L-GPIO4_A2_D-PadY4) -> GMAC1_RXD3_M1
- U1 pad Y5: unconnected-(U1L-GPIO3_D7_D-PadY5) -> Net-(U1L-GPIO3_D7_D)
- U1 pad Y6: unconnected-(U1L-GPIO3_D6_D-PadY6) -> Net-(U1L-GPIO3_D6_D)
- U36 pad 13: GMAC0_MDC -> GMAC1_MDC_M1
- U36 pad 14: GMAC0_MDIO -> GMAC1_MDIO_M1
- U36 pad 15: GMAC0_TXD3 -> GMAC1_TXD3_M1
- U36 pad 16: GMAC0_TXD2 -> GMAC1_TXD2_M1
- U36 pad 17: GMAC0_TXD1 -> GMAC1_TXD1_M1
- U36 pad 18: GMAC0_TXD0 -> GMAC1_TXD0_M1
- U36 pad 19: GMAC0_TXEN -> GMAC1_TXEN_M1
- U36 pad 20: GMAC0_TXCLK -> GMAC1_TXCLK_M1
- U46 pad 1: GND -> /PCIE/PI6C_03_S0
- U46 pad 2: MIC1_INP -> /PCIE/PI6C_03_S1
- U57 pad 3: ALPS_INT_L_GPIO2_D3 -> HALL_INT_L_GPIO0_C6
- U6 pad 3: /Power/USB3_OTG0_SSTXP -> USB3_OTG0_SSTXP
- U6 pad 4: /Power/USB3_OTG0_SSTXN -> USB3_OTG0_SSTXN
- U6 pad 9: /Power/TYPEC_0_SW_SEL_GPIO4_D2 -> TYPEC_SW_SEL_GPIO4_D2
- U7 pad 5: /Power/USBCC_INT_L_GPIO0_C5 -> USBCC_INT_L_GPIO0_C5
- U8 pad 7: /Power/CHG_INT_L_GPIO0_C2 -> CHG_INT_L_GPIO0_C2
- U8 pad 8: /Power/BQ_OTG_EN_H_GPIO3_C3 -> BQ_OTG_EN_H_GPIO3_C3
Routing:
- net LPDDR4_CLKP_A: track 0.00 -> 0.57 mm
