File: hardware/board/frost.kicad_pcb (KiCad board)
At the start: 2 copper layers, 90 x 55 mm, 739 parts, among them CN1 PJ-393 8PJ, CN2 1-2199230-5, J1 HDMI_A, J4 Conn_01x04, Q1 WPM3407-3/TR, Q2 SS8050, Q3 WPM2015-3/TR_C7472861, Q4 WPM2015-3/TR_C7472861, Q5 SS8050, Q6 2SK3018_C194460, Q7 2SK3018_C194460, Q8 2SK3018_C194460, Q9 WPM2015-3/TR_C7472861, SW1 TS24CA, SW2 TS24CA, SW3 TS24CA, U1 RK3568, U10 SY8088AAC, U11 RK860-0, U12 SY7208ABC, U13 FTC252012SR24MBCA, U14 ESD5311X, U15 ESD5311X, U16 ESD5311X, U17 ESD5311X, U18 SY6280AAC, U19 ESD5311X, U2 K4UCE3Q4AB-MGCL, U20 ESD5311X, U21 ESD5311X, U22 ESD5311X, U23 ESD5311X, U24 ESD5311X, U25 ESD5311X, U26 LP3983SAB5F-08, U27 5054133410_C6422029, U28 ESD5341N, U29 ESD5341N, U3 KLMBG2JETD-B041_C5821038, U30 ESD5341N, U31 ESD5341N, U32 SY7203DBC, U33 CY54-4.7UH, U34 AP6275PR3, U35 TFM252012ALVA2R2MTAA, U36 RTL8211F-CG, U37 TFM252012ALVA2R2MTAA, U38 ESD5451N_C5261080, U39 ESD5451N_C5261080, U4 RK809-5, U40 ESD5451N_C5261080, U41 ESD5451N_C5261080, U42 ESD5451N_C5261080, U43 ESD5451N_C5261080, U44 ESD5451N_C5261080, U45 ESD5451N_C5261080, U46 PI6C557-03BLE, U47 ESD5451N_C5261080, U48 ESD5451N_C5261080, U49 ESD5451N_C5261080, U5 TFM252012ALVA2R2MTAA, U50 TP5108E23E-33, U51 SY8089AAAC, U52 MXC6655XA, U53 AK09918C, U54 SC7A20TR_C5126709, U55 ICM-20600, U56 STK3311-X_C966926, U57 HAL248TDSO, U58 ESD5451N_C5261080, U59 ESD5451N_C5261080, U6 TMUXHS4212RKSR, U60 ESD5451N_C5261080, U61 ESD5451N_C5261080, U62 ESD5451N_C5261080, U7 FUSB302BMPX, U8 BQ25890RTWR, U9 S2B-PH-K-S(LF)(SN), X1 24 MHz, X2 Q13FC1350000400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

Commit message: did a thing
Parts:
- removed the C198 at (181.5, -3.47)
- removed the C198 at (174.2, -26.8)
- removed the C199 at (154.4, -26.8)
- removed the C199 at (181.5, -1.50)
- removed the C2 at (180.9, 109.4)
- removed the C2 at (209.0, 121.5)
- removed the CN2 at (109.3, 135.6)
- removed the CN2 at (219.5, 3.15)
- removed D2, D3, D4, D5: BZT52C5V1_C173407, lcsc:SOD-123_L2.7-W1.6-LS3.7-RD
- removed the R1 at (206.1, 121.5)
- removed the R1 at (186.4, 102.7)
- removed R113, R114, R117, R122, R124, R125: 4.7K 5%, Resistor_SMD:R_0402_1005Metric
- removed the R129 at (171.3, -26.8)
- removed the R129 at (178.6, -3.46)
- removed the R139 at (178.6, -1.47)
- removed the R139 at (171.3, -24.8)
- removed R168, R170: 10K 5%, Resistor_SMD:R_0402_1005Metric
- removed R191: 100K 5%, Resistor_SMD:R_0402_1005Metric
- removed the R2 at (186.4, 104.7)
- removed the R2 at (206.1, 123.5)
- removed R60, R61: 0R 5%, Resistor_SMD:R_0402_1005Metric
- removed the U46 at (256.6, 44.3)
- removed the U46 at (219.5, -18.1)
- added C198: 100nF X5R 10V, Capacitor_SMD:C_0402_1005Metric, F.Cu at (138.1, 151.3)
- added C199: 100nF X5R 10V, Capacitor_SMD:C_0402_1005Metric, F.Cu at (107.5, 47.1)
- added C2: 10pF C0G 50V, Capacitor_SMD:C_0402_1005Metric, F.Cu at (138.1, 149.4)
- added CN2: 1-2199230-5, lcsc:PCIE-SMD_75P-P0.50_1-2199230-5, F.Cu at (122.8, 116.3)
- added J3: USB3_A, lcsc:USB-A-SMD_U-A-39SS-W-1, F.Cu at (74.5, 137.7)
- added R1: 22R 5%, Resistor_SMD:R_0402_1005Metric, F.Cu at (148.4, 146.8)
- added R129: 1K 5%, Resistor_SMD:R_0402_1005Metric, F.Cu at (148.4, 150.8)
- added R139: 100K 5%, Resistor_SMD:R_0402_1005Metric, F.Cu at (148.4, 152.8)
- added R2: 1M 5%, Resistor_SMD:R_0402_1005Metric, F.Cu at (148.4, 148.8)
- added U46: PI6C557-03BLE, lcsc:TSSOP-16_L5.0-W4.4-P0.65-LS6.4-BL, F.Cu at (79.5, 212.9)
- added U63: SY8089AAAC, lcsc:SOT-23-5_L3.0-W1.7-P0.95-LS2.8-BR, F.Cu at (-56.0, 99.8)
- added U64: FTC252012SR47MBCA, lcsc:IND-SMD_L2.5-W2.0, F.Cu at (111.1, 45.1)
- added U65: FTC252012SR47MBCA, lcsc:IND-SMD_L2.5-W2.0, F.Cu at (111.1, 48.4)
- added U66: FTC252012SR47MBCA, lcsc:IND-SMD_L2.5-W2.0, F.Cu at (111.1, 51.7)
- added U67: FTC252012SR47MBCA, lcsc:IND-SMD_L2.5-W2.0, F.Cu at (111.1, 55.0)
- added U68: ESD5341N, lcsc:DFN1006-2L-RD, B.Cu at (-41.4, 67.2)
- added U69: ESD5341N, lcsc:DFN1006-2L-RD, B.Cu at (-42.4, 67.2)
- added U70: ESD5341N, lcsc:DFN1006-2L-RD, B.Cu at (-42.4, 63.8)
- added U71: ESD5341N, lcsc:DFN1006-2L-RD, B.Cu at (-41.2, 63.8)
- added USBC1: 105450-0101, lcsc:USB-C-SMD_TYPE-C-USB-18, F.Cu at (-41.9, 67.0)
- C11, C12, C13, C14: footprint Capacitor_SMD:C_0402_1005Metric -> Capacitor_SMD:C_0201_0603Metric
- C309, C310, C311, R156, U9: moved to B.Cu
- R94: value 0R 5% -> 22R 5%
- U10: value SY8088AAC -> FTC252012SR47MBCA; footprint lcsc:SOT-23-5_L3.0-W1.7-P0.95-LS2.8-BR -> lcsc:IND-SMD_L2.5-W2.0
- moved Q3 298.0 mm to (-107.8, 62.4)
- moved R30 285.9 mm to (-108.6, 63.4)
- moved R29 285.0 mm to (-107.3, 64.5)
- moved Q2 277.8 mm to (-86.6, 96.7), turned to 180 degrees
- moved C37 272.1 mm to (-86.5, 100.2), turned to 90 degrees
- moved L3 271.6 mm to (-83.5, 104.5)
- moved D9 271.5 mm to (-79.1, 102.8), turned to -90 degrees
- moved R23 271.0 mm to (-90.7, 99.7), turned to 90 degrees
- moved R26 269.2 mm to (-83.1, 98.2), turned to -90 degrees
- moved U12 268.7 mm to (-83.2, 100.8)
- moved R24 268.1 mm to (-88.6, 97.8), turned to 180 degrees
- moved R28 267.2 mm to (-82.2, 98.2), turned to -90 degrees
- moved R27 266.2 mm to (-80.7, 97.8)
- moved C42 263.8 mm to (-105.6, 62.3), turned to -90 degrees
- moved R25 263.3 mm to (-84.1, 98.2), turned to -90 degrees
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Connections:
- C32 pad 1: Net-(U10-EN) -> Net-(U63-EN)
- C33 pad 2: Net-(U10-FB) -> Net-(U63-FB)
- D7 pad 1: /Power/TYPEC_0_SSTX2P -> /Power/TYPEC_0_SSTX2N
- D7 pad 10: /Power/TYPEC_0_SSTX2P -> /Power/TYPEC_0_SSTX2N
- D7 pad 2: /Power/TYPEC_0_SSTX2N -> /Power/TYPEC_0_SSTX2P
- D7 pad 4: /Power/TYPEC_0_SSRX2P -> /Power/TYPEC_0_SSRX2N
- D7 pad 5: /Power/TYPEC_0_SSRX2N -> /Power/TYPEC_0_SSRX2P
- D7 pad 6: /Power/TYPEC_0_SSRX2N -> /Power/TYPEC_0_SSRX2P
- D7 pad 7: /Power/TYPEC_0_SSRX2P -> /Power/TYPEC_0_SSRX2N
- D7 pad 9: /Power/TYPEC_0_SSTX2N -> /Power/TYPEC_0_SSTX2P
- L1 pad 1: Net-(L1-Pad1) -> /Power/TYPEC_0_DP
- L1 pad 3: Net-(L1-Pad3) -> /Power/TYPEC_0_DM
- L4 pad 1: Net-(U10-LX) -> Net-(U63-LX)
- R20 pad 1: Net-(U10-EN) -> Net-(U63-EN)
- R21 pad 1: Net-(U10-FB) -> Net-(U63-FB)
- R22 pad 2: Net-(U10-FB) -> Net-(U63-FB)
- R7 pad 1: Net-(L1-Pad1) -> /Power/TYPEC_0_DP
- R8 pad 1: Net-(L1-Pad3) -> /Power/TYPEC_0_DM
- U1 pad P28: USB3_OTG0_DP -> USB3_OTG0_DM
- U1 pad R27: USB3_OTG0_SSRXP -> USB3_OTG0_SSRXN
- U1 pad R28: USB3_OTG0_SSRXN -> USB3_OTG0_SSRXP
- U1 pad T27: USB3_OTG0_SSTXP -> USB3_OTG0_SSTXN
- U1 pad T28: USB3_OTG0_SSTXN -> USB3_OTG0_SSTXP
- U1 pad U27: USB3_HOST1_SSRXP -> USB3_HOST1_SSRXN
- U1 pad U28: USB3_HOST1_SSRXN -> USB3_HOST1_SSRXP
- U1 pad V27: USB3_HOST1_SSTXP -> USB3_HOST1_SSTXN
- U1 pad V28: USB3_HOST1_SSTXN -> USB3_HOST1_SSTXP
- U10 pad 1: Net-(U10-EN) -> VDD_GPU
- U10 pad 2: unconnected-(U10-GND-Pad2) -> Net-(U4-SW2)
Routing:
- net /Power/TYPEC_0_SSTX2N: track 0.00 -> 7.70 mm, vias 0 -> 2
- net /Power/TYPEC_0_DM: track 0.00 -> 6.05 mm
- net /Power/TYPEC_0_DP: track 0.00 -> 6.05 mm
- net /Power/TYPEC_0_SSTX2P: track 0.00 -> 5.63 mm, vias 0 -> 2
- net /Power/TYPEC_0_SSRX1P: track 0.00 -> 5.63 mm, vias 0 -> 2
- net /Power/TYPEC_0_SSRX1N: track 0.00 -> 4.57 mm, vias 0 -> 2
- net Net-(U8-TS): track 0.00 -> 4.27 mm
- net Net-(U8-~{CE}): track 0.00 -> 3.24 mm
- net /Power/TYPEC_0_SSTX1P: track 0.00 -> 3.18 mm
- net /Power/TYPEC_0_SSTX1N: track 0.00 -> 3.18 mm
- net /Power/TYPEC_0_SSRX2P: track 0.00 -> 3.18 mm
- net /Power/TYPEC_0_SSRX2N: track 0.00 -> 3.18 mm
- net /Power/TYPEC_0_CC1: track 0.00 -> 2.89 mm, vias 0 -> 1
- net Net-(C25-Pad1): track 0.00 -> 2.23 mm
- net CHG_REF: track 0.00 -> 1.97 mm
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Other:
- board size 90 x 55 mm -> 91 x 56 mm
- copper layers 2 -> 6
