File: hardware/board/frost.kicad_pcb (KiCad board)
At the start: 6 copper layers, 91 x 56 mm, 726 parts, among them CN1 PJ-393 8PJ, CN2 1-2199230-5, J1 HDMI_A, J3 USB3_A, J4 Conn_01x04, Q1 WPM3407-3/TR, Q2 SS8050, Q3 WPM2015-3/TR_C7472861, Q4 WPM2015-3/TR_C7472861, Q5 SS8050, Q6 2SK3018_C194460, Q7 2SK3018_C194460, Q8 2SK3018_C194460, Q9 WPM2015-3/TR_C7472861, SW1 TS24CA, SW2 TS24CA, SW3 TS24CA, U1 RK3568, U10 FTC252012SR47MBCA, U11 RK860-0, U12 SY7208ABC, U13 FTC252012SR24MBCA, U14 ESD5311X, U15 ESD5311X, U16 ESD5311X, U17 ESD5311X, U18 SY6280AAC, U19 ESD5311X, U2 K4UCE3Q4AB-MGCL, U20 ESD5311X, U21 ESD5311X, U22 ESD5311X, U23 ESD5311X, U24 ESD5311X, U25 ESD5311X, U26 LP3983SAB5F-08, U27 5054133410_C6422029, U28 ESD5341N, U29 ESD5341N, U3 KLMBG2JETD-B041_C5821038, U30 ESD5341N, U31 ESD5341N, U32 SY7203DBC, U33 CY54-4.7UH, U34 AP6275PR3, U35 TFM252012ALVA2R2MTAA, U36 RTL8211F-CG, U37 TFM252012ALVA2R2MTAA, U38 ESD5451N_C5261080, U39 ESD5451N_C5261080, U4 RK809-5, U40 ESD5451N_C5261080, U41 ESD5451N_C5261080, U42 ESD5451N_C5261080, U43 ESD5451N_C5261080, U44 ESD5451N_C5261080, U45 ESD5451N_C5261080, U46 PI6C557-03BLE, U47 ESD5451N_C5261080, U48 ESD5451N_C5261080, U49 ESD5451N_C5261080, U5 TFM252012ALVA2R2MTAA, U50 TP5108E23E-33, U51 SY8089AAAC, U52 MXC6655XA, U53 AK09918C, U54 SC7A20TR_C5126709, U55 ICM-20600, U56 STK3311-X_C966926, U57 HAL248TDSO, U58 ESD5451N_C5261080, U59 ESD5451N_C5261080, U6 TMUXHS4212RKSR, U60 ESD5451N_C5261080, U61 ESD5451N_C5261080, U62 ESD5451N_C5261080, U63 SY8089AAAC, U64 FTC252012SR47MBCA, U65 FTC252012SR47MBCA, U66 FTC252012SR47MBCA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

Commit message: more stuff
Parts:
- moved RJ1 162.0 mm to (-7.61, 246.8), turned to -90 degrees
- moved C194 151.2 mm to (13.3, 260.4)
- moved C195 151.2 mm to (16.2, 248.6)
- moved C196 151.2 mm to (16.2, 250.6)
- moved C197 151.2 mm to (16.2, 252.5)
- moved R131 151.2 mm to (16.5, 228.7)
- moved R132 151.2 mm to (16.5, 230.7)
- moved R133 151.2 mm to (16.5, 232.7)
- moved R134 151.2 mm to (16.5, 234.7)
- moved R135 151.2 mm to (16.5, 236.7)
- moved R136 151.2 mm to (16.5, 238.7)
- moved R137 151.2 mm to (16.5, 240.6)
- moved R138 151.2 mm to (16.5, 242.6)
- moved FB11 151.2 mm to (19.6, 258.9)
- moved R110 151.2 mm to (10.7, 228.7)
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Routing:
- net GND: track 1.42 -> 4.29 mm
