File: hardware/board/power.kicad_sch (KiCad schematic)
At the start: 180 parts, among them J2 USB_C_Receptacle, Q1 WPM3407-3/TR, Q2 SS8050, Q3 WPM2015-3/TR_C7472861, U10 SY8088AAC, U12 SY7208ABC, U4 RK809-5, U6 TMUXHS4212RKSR, U7 FUSB302BMPX, U8 BQ25890RTWR, U9 S2B-PH-K-S(LF)(SN), X2 Q13FC1350000400

Commit message: emmc stuff
Parts:
- added C102, C103: 22uF X5R 10V, Capacitor_SMD:C_0805_2012Metric, symbol Device:C
- added C104, C105, C106: 22uF X5R 6.3V, Capacitor_SMD:C_0603_1608Metric, symbol Device:C
- added C107, C108, C109, C110, C111, C115, C116: 1uF X5R 6.3V, Capacitor_SMD:C_0402_1005Metric, symbol Device:C
- added C112, C114: 10uF X5R 10V, Capacitor_SMD:C_0603_1608Metric, symbol Device:C
- added C113: 100nF X5R 10V, Capacitor_SMD:C_0402_1005Metric, symbol Device:C
- added C117: 4.7uF X5R 6.3V, Capacitor_SMD:C_0603_1608Metric, symbol Device:C
- added FB10, FB7, FB8, FB9: 120@100MHz 0.03R, Inductor_SMD:L_0603_1608Metric, symbol Device:FerriteBead
- added Q4: WPM2015-3/TR_C7472861, lcsc:SOT-23-3_L2.9-W1.3-P1.90-LS2.4-BR, symbol lcsc:WPM2015-3_TR_C7472861
- added Q5: SS8050, Package_TO_SOT_SMD:SOT-23, symbol Transistor_BJT:SS8050
- added R48, R52: 51K 5%, Resistor_SMD:R_0402_1005Metric, symbol Device:R
- added R49: 100R 5%, Resistor_SMD:R_0402_1005Metric, symbol Device:R
- added R50: 100K 5%, Resistor_SMD:R_0402_1005Metric, symbol Device:R
- added R51, R53, R57: 10K 5%, Resistor_SMD:R_0402_1005Metric, symbol Device:R
- added R54, R55, R56, R60, R61: 0R 5%, Resistor_SMD:R_0402_1005Metric, symbol Device:R
- added U11: RK860-0, lcsc:WLCSP-20_L2.0-W1.6-R5-C4-P0.40-TL, symbol lcsc:RK860-0
- added U13: FTC252012SR24MBCA, lcsc:IND-SMD_L2.5-W2.0_MHCHL2520, symbol lcsc:FTC252012SR24MBCA
- R7, R8: value 2.2R -> 2.2R 5%; footprint Resistor_SMD:R_1206_3216Metric -> Resistor_SMD:R_0402_1005Metric
Connections:
- net GND: now also C102.2, C103.2, C104.2, C105.2, C106.2, C108.2, C109.2, C110.2, C111.2, C112.2, C114.2, C115.2, C116.2, C117.2, Q5.2 (E), R52.1, U11.B2 (GND), U11.B3 (GND), U11.B4 (AGND), U11.C1 (GND), U11.C2 (GND), U11.C3 (GND), U11.C4 (GND)
- net I2C0_SCL_PMIC: now also U11.A3 (SCL)
- net I2C0_SDA_PMIC: now also U11.B1 (SDA)
- net PMIC_SLEEP_H: now also U11.A1 (VSEL)
- net TYPEC_0_DP: now also R60.1
- net USB3_OTG0_DP: no longer R8.2
- net VCC3V3_PMU: now also R48.2, R57.2
- net VCC3V3_SYS: now also C112.1, C113.1, Q4.2 (S), R50.2
- net VCCA1V8_PMU: now also R54.2
- net VCCA_1V8: now also C109.1, FB8.1
- net VCC_1V8: now also R56.2
- net VCC_SYSIN: now also C102.1, C103.1, U11.D1 (VIN), U11.D2 (VIN), U11.E1 (VIN), U11.E2 (VIN)
- net VDDA0V9_IMAGE: now also C110.1, FB9.1
- net VDDA_0V9: now also C108.1, FB7.1
- net at L1.1, R7.1: now also R60.2
- net at L1.3, R8.1: now also R61.1
- net TYPEC_0_DN renamed TYPEC_0_DM
- net TYPEC_0_DM: now also R61.2
- new net: Q5.3 (C), R51.1
- new net: C113.2, Q4.1 (G), R50.1, R51.2
- new net: Q5.1 (B), R52.2, R53.1
- new net: R48.1, U11.A2 (EN)
- new net: U11.D3 (LX), U11.D4 (LX), U11.E3 (LX), U11.E4 (LX), U13.1
- new net FLASH_VOL_SEL: R57.1
- new net LCD0_PWREN_H_GPIO0_C7: R53.2
- new net MIPI_AVDD_0V9: FB9.2
- new net MIPI_AVDD_1V8: FB10.2
- new net PMUIO2: C115.1, R54.1, R55.2
- new net USB3_OTG0_DM: R8.2
- new net USB_AVDD_0V9: FB7.2
- new net USB_AVDD_1V8: FB8.2
- new net VCC3V3_LCD0: C114.1, Q4.3 (D)
- new net VCCA1V8_IMAGE: C111.1, FB10.1
- new net VCCIO_FLASH: C117.1, R56.1
- new net VCCIO_WL: C116.1, R55.1
- new net VDD_CPU: C104.1, C105.1, C106.1, C107.2, R49.1, U13.2
- new net VDD_CPU_COM: C107.1, R49.2, U11.A4 (VOUT)
Other:
- note added: "Charger IC"
- note added: "Differential Channel Crossbar Switch"
- note added: "FLASH"
- note added: "LCD Power"
- note added: "Note: FLASH_VOL_SEL is pulled up if 1.8v and down if 3.3v"
- note added: "PMIC RK809"
- note added: "Peripheral power input source"
- note added: "USB Type-C Controller(PD)"
- note added: "USB-C / ESD"
- note added: "USB/MIPI PHY Power"
- note added: "VCC/VDDA"
- note added: "VCC3V3_SYS"
- note added: "VCC_3V3 (OFF under SLEEP)"
- note added: "VCC_5V0"
- note added: "VDD_CPU"
- note added: "WIFI/BT IO and CTL IO Power"
- moved on the sheet: C10, C11, C12, C13, C14, C15, C16, C17, C18, C19, C20, C36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

Commit message: start of ethernet
Connections:
- net VCCA1V8_IMAGE: now also C48.1, FB3.2
- net VCC_1V8: no longer C48.1, FB3.2
Changed lines of the file:
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@@
 			)
 		)
-		(property "Value" "VCC_1V8"
+		(property "Value" "VCCA1V8_IMAGE"
 			(at 279.4 363.982 0)
 			(effects

Commit message: add in pcie and ddr4
Parts:
- added C199: 100nF X5R 10V, Capacitor_SMD:C_0402_1005Metric, symbol Device:C
- added C254, C261, C264: 4.7uF X5R 6.3V, Capacitor_SMD:C_0402_1005Metric, symbol Device:C
- added C255, C256, C257, C259, C260, C263, C269, C271, C272: 22uF X5R 6.3V, Capacitor_SMD:C_0603_1608Metric, symbol Device:C
- added C258, C268, C273: 10uF X5R 6.3V, Capacitor_SMD:C_0603_1608Metric, symbol Device:C
- added C262, C265, C270: 100nF X5R 10V, Capacitor_SMD:C_0201_0603Metric, symbol Device:C
- added C266, C267: 1uF X5R 6.3V, Capacitor_SMD:C_0402_1005Metric, symbol Device:C
- added U1: RK3568, RK3568:BGA636C65P28X28_1900X1900X168, symbol RK3568:RK3568
Connections:
- net VDD_CPU: now also C199.1, C254.1, C255.1, C256.1, C257.1, U1.J15 (VDD_CPU), U1.K15 (VDD_CPU), U1.K16 (VDD_CPU), U1.K17 (VDD_CPU), U1.K18 (VDD_CPU), U1.L15 (VDD_CPU), U1.L16 (VDD_CPU), U1.L17 (VDD_CPU), U1.L18 (VDD_CPU), U1.M17 (VDD_CPU)
- net VDD_CPU_COM: now also U1.M15 (VDD_CPU_COM)
- net VDD_GPU: now also C258.1, C259.1, C260.1, C261.1, C262.1, U1.R13 (VDD_GPU), U1.T13 (VDD_GPU), U1.U11 (VDD_GPU), U1.U12 (VDD_GPU), U1.U13 (VDD_GPU)
- net VDD_LOGIC: now also C263.1, C264.1, C265.1, C266.1, C267.1, C268.1, C269.1, U1.L12 (VDD_LOGIC), U1.M12 (VDD_LOGIC), U1.N13 (VDD_LOGIC), U1.N16 (VDD_LOGIC), U1.P13 (VDD_LOGIC), U1.P16 (VDD_LOGIC), U1.R12 (VDD_LOGIC), U1.R16 (VDD_LOGIC), U1.T12 (VDD_LOGIC), U1.T16 (VDD_LOGIC)
- net VDD_NPU: now also C270.1, C271.1, C272.1, C273.1, U1.M19 (VDD_NPU), U1.N19 (VDD_NPU), U1.P18 (VDD_NPU), U1.P19 (VDD_NPU), U1.P20 (VDD_NPU)
- net GND renamed AVSS1
- net AVSS1: now also C199.2, C254.2, C255.2, C256.2, C257.2, C258.2, C259.2, C260.2, C261.2, C262.2, C263.2, C264.2, C265.2, C266.2, C267.2, C268.2, C269.2, C270.2, C271.2, C272.2, C273.2, U1.A1 (VSS1), U1.A10 (VSS1), U1.A14 (VSS1), U1.A18 (VSS1), U1.A28 (VSS1), U1.A3 (VSS1), U1.A6 (VSS1), U1.AA12 (AVSS2), U1.AA14 (AVSS2), U1.AA15 (AVSS2), U1.AA17 (AVSS2), U1.AA23 (VSS9), U1.AA24 (AVSS2), U1.AA26 (AVSS2), U1.AA4 (VSS9), U1.AA9 (VSS9), U1.AB11 (AVSS2), U1.AB12 (AVSS3), U1.AB14 (AVSS3), U1.AB15 (AVSS3), U1.AB17 (AVSS3), U1.AB2 (VSS10), U1.AB6 (VSS10), U1.AC11 (AVSS3), U1.AC12 (AVSS3), U1.AC15 (AVSS3), U1.AC18 (AVSS3), U1.AC25 (AVSS3), U1.AC26 (AVSS3), U1.AC9 (AVSS3), U1.AD26 (AVSS3), U1.AD3 (VSS10), U1.AE14 (AVSS3), U1.AE17 (AVSS3), U1.AE20 (AVSS3), U1.AE21 (VSS10), U1.AE27 (AVSS4), U1.AE28 (AVSS4), U1.AE6 (VSS10), U1.AF11 (AVSS4), U1.AF12 (AVSS4), U1.AF14 (AVSS4), U1.AF15 (AVSS4), U1.AF17 (AVSS4), U1.AF18 (AVSS4), U1.AF20 (AVSS4), U1.AF21 (AVSS4), U1.AF26 (VSS10), U1.AF3 (VSS10), U1.AF9 (AVSS4), U1.AG18 (AVSS4), U1.AG5 (VSS10), U1.AH1 (VSS10), U1.AH18 (AVSS4), U1.AH23 (AVSS4), U1.AH28 (VSS10), U1.AH8 (VSS10), U1.B12 (VSS1), U1.B16 (VSS1), U1.B23 (VSS1), U1.B26 (VSS1), U1.B5 (VSS1), U1.B9 (VSS1), U1.C11 (VSS2), U1.C12 (VSS2), U1.C14 (VSS2), U1.C15 (VSS2), U1.C17 (VSS2), U1.C18 (VSS2), U1.C25 (VSS2), U1.C3 (VSS1), U1.C6 (VSS1), U1.C8 (VSS2), U1.C9 (VSS2), U1.D11 (VSS2), U1.D2 (VSS2), U1.D28 (VSS2), U1.D3 (VSS2), U1.E3 (VSS2), U1.E7 (VSS2), U1.F1 (VSS3), U1.F12 (VSS3), U1.F14 (VSS3), U1.F15 (VSS3), U1.F17 (VSS3), U1.F3 (VSS3), U1.F9 (VSS3), U1.G11 (VSS3), U1.G12 (VSS3), U1.G14 (VSS3), U1.G15 (VSS3), U1.G17 (VSS4), U1.G18 (VSS4), U1.G24 (VSS4), U1.G5 (VSS3), U1.G6 (VSS3), U1.G8 (VSS3), U1.G9 (VSS3), U1.H2 (VSS4), U1.H3 (VSS4), U1.H6 (VSS4), U1.J17 (VSS4), U1.J18 (VSS4), U1.J20 (VSS4), U1.J22 (VSS4), U1.J26 (VSS4), U1.J27 (AVSS1), U1.J3 (VSS4), U1.J5 (VSS4), U1.K1 (VSS4), U1.K11 (VSS4), U1.K12 (VSS5), U1.K13 (VSS5), U1.K14 (VSS5), U1.K19 (VSS5), U1.L11 (VSS5), U1.L13 (VSS5), U1.L14 (VSS5), U1.L19 (VSS5), U1.L20 (VSS5), U1.L21 (VSS5), U1.L24 (AVSS1), U1.L26 (AVSS1), U1.L3 (VSS5), U1.L5 (VSS5), U1.L8 (VSS5), U1.M11 (VSS6), U1.M13 (VSS6), U1.M14 (VSS6), U1.M16 (VSS6), U1.M18 (VSS6), U1.M2 (VSS5), U1.M21 (AVSS1), U1.M26 (AVSS1), U1.M3 (VSS5), U1.M6 (VSS6), U1.M8 (VSS6), U1.N1 (VSS6), U1.N12 (VSS6), U1.N14 (VSS6), U1.N15 (VSS6), U1.N17 (VSS6), U1.N18 (VSS6), U1.N28 (AVSS1), U1.P12 (VSS7), U1.P14 (VSS7), U1.P15 (VSS7), U1.P17 (VSS7), U1.P21 (AVSS1), U1.P26 (AVSS1), U1.P3 (VSS6), U1.P6 (VSS6), U1.R10 (VSS7), U1.R11 (VSS7), U1.R14 (VSS7), U1.R15 (VSS7), U1.R17 (VSS7), U1.R18 (VSS7), U1.R19 (VSS7), U1.R23 (AVSS1), U1.R26 (AVSS1), U1.R3 (VSS7), U1.R6 (VSS7), U1.T10 (VSS7), U1.T11 (VSS7), U1.T14 (VSS8), U1.T15 (VSS8), U1.T17 (VSS8), U1.T18 (VSS8), U1.T19 (VSS8), U1.U1 (VSS8), U1.U10 (VSS8), U1.U14 (VSS8), U1.U15 (VSS8), U1.U16 (VSS8), U1.U17 (VSS8), U1.U18 (VSS8), U1.U23 (AVSS1), U1.U26 (AVSS1), U1.U6 (VSS8), U1.U7 (VSS8), U1.U8 (VSS8), U1.V13 (VSS9), U1.V14 (AVSS1), U1.V15 (AVSS1), U1.V16 (AVSS1), U1.V22 (AVSS2), U1.V23 (AVSS2), U1.V26 (AVSS2), U1.V3 (VSS9), U1.V8 (VSS9), U1.V9 (VSS9), U1.W10 (VSS9), U1.W11 (VSS9), U1.W12 (VSS9), U1.W13 (VSS9), U1.W17 (AVSS2), U1.Y11 (VSS9), U1.Y12 (VSS9), U1.Y18 (AVSS2), U1.Y23 (AVSS2), U1.Y24 (AVSS2), U1.Y26 (AVSS2), U1.Y8 (VSS9), U1.Y9 (VSS9)
Other:
- note added: "RK3568"
- note added: "Should be placed close"
- note added: "Should be placed under"
- moved on the sheet: C10, C100, C101, C11, C12, C13, C14, C50, C51, C52, C53, C54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
