File: hardware/board/power.kicad_sch (KiCad schematic)
At the start: 238 parts, among them J2 USB_C_Receptacle, Q1 WPM3407-3/TR, Q2 SS8050, Q3 WPM2015-3/TR_C7472861, Q4 WPM2015-3/TR_C7472861, Q5 SS8050, U1 RK3568, U10 SY8088AAC, U11 RK860-0, U12 SY7208ABC, U13 FTC252012SR24MBCA, U4 RK809-5, U6 TMUXHS4212RKSR, U7 FUSB302BMPX, U8 BQ25890RTWR, U9 S2B-PH-K-S(LF)(SN), X2 Q13FC1350000400

Commit message: finished schematic!
Parts:
- added C334, C336: 10uF X5R 10V, Capacitor_SMD:C_0603_1608Metric, symbol Device:C
- added C335: 100nF X5R 10V, Capacitor_SMD:C_0402_1005Metric, symbol Device:C
- added C372: 100nF X5R 10V, Capacitor_SMD:C_0201_0603Metric, symbol Device:C
- added Q9: WPM2015-3/TR_C7472861, lcsc:SOT-23-3_L2.9-W1.3-P1.90-LS2.4-BR, symbol lcsc:WPM2015-3_TR_C7472861
- added R190: 10K 5%, Resistor_SMD:R_0402_1005Metric, symbol Device:R
- added R191, R192: 100K 5%, Resistor_SMD:R_0402_1005Metric, symbol Device:R
- added R220, R221, R223, R224: 22R 5%, Resistor_SMD:R_0402_1005Metric, symbol Device:R
- added unit 7 of U1
Connections:
- net AVSS1: now also C334.2, C336.2, C372.2, R191.1; no longer C42.2
- net I2S1_LRCK_TX_M0_PMIC: now also R223.2
- net I2S1_MCLK_M0_PMIC: now also R220.2
- net I2S1_SCLK_TX_M0_PMIC: now also R221.2
- net I2S1_SDI0_M0/PDM_SDI0_M0_PMIC: now also U1.B21 (GPIO1_B3_D)
- net I2S1_SDO0_M0_PMIC: now also U1.B20 (GPIO1_A7_D)
- net PDM_CLK0_M0_PMIC: now also R224.2
- net VCC3V3_SD: now also C336.1, Q9.3 (D)
- net VCC3V3_SYS: now also C334.1, C335.1, Q9.2 (S), R192.2
- net VCCIO_ACODEC: now also C372.1, U1.H17 (VCCIO1)
- net at Q3.1 (G), R29.2: now also C42.2
- net TYPEC_0_SW_SEL_GPIO4_D2 renamed TYPEC_SW_SEL_GPIO4_D2
- new net: R224.1, U1.C20 (GPIO1_A6_D)
- new net: C335.2, Q9.1 (G), R190.2, R192.1
- new net: R221.1, U1.B19 (GPIO1_A3_D)
- new net: R220.1, U1.A19 (GPIO1_A2_D)
- new net: R223.1, U1.A20 (GPIO1_A5_D)
- new net SDMMC0_PWREN_L: R190.1, R191.2
- no-connect marks 9 -> 15
Other:
- note added: "I2C if needed"
- note added: "VCC_3V3_SD"
- moved on the sheet: C102, C103, C104, C105, C106, C107, C115, C116, C41, C42, C44, C45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

Commit message: finished beautifying schematic
Other:
- note added: "Frost"
- note added: "Power"
- note added: "Power Schematics"
- note added: "USB-C PD"
- note removed: "USB Type-C Controller(PD)"
- moved on the sheet: C10, C100, C101, C102, C103, C104, C105, C106, C107, C108, C109, C11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

Commit message: did a thing
Parts:
- removed D2, D3, D4, D5: BZT52C5V1_C173407, lcsc:SOD-123_L2.7-W1.6-LS3.7-RD, symbol lcsc:BZT52C5V1_C173407
- removed J2: USB_C_Receptacle, symbol Connector:USB_C_Receptacle
- removed L5, L6, L7, L8, L9: 470nH, symbol Device:L
- removed R60, R61: 0R 5%, Resistor_SMD:R_0402_1005Metric, symbol Device:R
- removed U10: SY8088AAC, lcsc:SOT-23-5_L3.0-W1.7-P0.95-LS2.8-BR, symbol lcsc:SY8088AAC
- added U10, U64, U65, U66, U67: FTC252012SR47MBCA, lcsc:IND-SMD_L2.5-W2.0, symbol lcsc:FTC252012SR47MBCA
- added U63: SY8089AAAC, lcsc:SOT-23-5_L3.0-W1.7-P0.95-LS2.8-BR, symbol lcsc:SY8089AAAC
- added U68, U69, U70, U71: ESD5341N, lcsc:DFN1006-2L-RD, symbol lcsc:ESD5341N
- added USBC1: 105450-0101, lcsc:USB-C-SMD_TYPE-C-USB-18, symbol lcsc:105450-0101
- C11, C12, C13, C14: footprint Capacitor_SMD:C_0402_1005Metric -> Capacitor_SMD:C_0201_0603Metric
Connections:
- net AVSS1: now also U68.2, U69.2, U70.2, U71.2, USBC1.0, USBC1.A1 (GND), USBC1.A12 (GND), USBC1.B1 (GND), USBC1.B12 (GND)
- net TYPEC_0_CC1: now also U69.1, USBC1.A5 (CC1)
- net TYPEC_0_CC2: now also U68.1, USBC1.B5 (CC2)
- net TYPEC_0_DM: now also L1.3, R8.1, U71.1, USBC1.A7 (D-), USBC1.B6 (D+)
- net TYPEC_0_DP: now also L1.1, R7.1, U70.1, USBC1.A6 (D+), USBC1.B7 (D-)
- net TYPEC_0_SSRX1N: now also USBC1.B10 (RX1-)
- net TYPEC_0_SSRX1P: now also USBC1.B11 (RX1+)
- net TYPEC_0_SSRX2N: now also D7.4, D7.7, USBC1.A10 (RX2-); no longer D7.5, D7.6
- net TYPEC_0_SSRX2P: now also D7.5, D7.6, USBC1.A11 (RX2+); no longer D7.4, D7.7
- net TYPEC_0_SSTX1N: now also USBC1.A3 (TX1-)
- net TYPEC_0_SSTX1P: now also USBC1.A2 (TX1+)
- net TYPEC_0_SSTX2N: now also D7.1, D7.10, USBC1.B3 (TX2-); no longer D7.2, D7.9
- net TYPEC_0_SSTX2P: now also D7.2, D7.9, USBC1.B2 (TX2+); no longer D7.1, D7.10
- net VBUS_TYPEC_0: now also USBC1.A4 (VBUS), USBC1.A9 (VBUS), USBC1.B4 (VBUS), USBC1.B9 (VBUS)
- net VCC_1V8: now also U66.2
- net VCC_DDR: now also U65.1
- net VCC_SYSIN: now also U63.4 (IN)
- net VDD_GPU: now also U10.1
- net VDD_LOGIC: now also U64.1
- net VDD_NPU: now also U67.2
- net at U4.12 (SW1): now also U64.2
- net at C32.1, R20.1: now also U63.1 (EN)
- net at L4.1: now also U63.3 (LX)
- net at C33.2, R21.1, R22.2: now also U63.5 (FB)
- net at U4.25 (SW3): now also U65.2
- net at U4.53 (SW5): now also U66.1
- net at U4.65 (SW4): now also U67.1
- net at U4.9 (SW2): now also U10.2
Other:
- moved on the sheet: C3, C4, C5, C58, C6, D1, D6, D7, L1, R3, R4, R5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
