File: hardware/board/memory_storage.kicad_sch (KiCad schematic)
At the start: 3 parts, among them U1 RK3568, U2 K4UCE3Q4AB-MGCL, U3 KLMBG2JETD-B041_C5821038

Commit message: emmc stuff
Parts:
- added C123: 2.2uF X5R 10V, Capacitor_SMD:C_0402_1005Metric, symbol Device:C
- added C124, C125, C126, C127, C128, C131, C132: 100nF X5R 10V, Capacitor_SMD:C_0402_1005Metric, symbol Device:C
- added C129, C130: 4.7uF X5R 6.3V, Capacitor_SMD:C_0603_1608Metric, symbol Device:C
- added R67, R68, R69: 10K 5%, Resistor_SMD:R_0402_1005Metric, symbol Device:R
- U1: LCSC (none) -> C3345225
Connections:
- net eMMC_D0: now reaches U3.A3 (DAT0)
- net eMMC_D0: now also R67.1
- net eMMC_D1: now reaches U3.A4 (DAT1)
- net eMMC_D2: now reaches U3.A5 (DAT2)
- net GND: now reaches U3.A6 (VSS)
- net GND: now also U3.C4 (VSS), U3.E7 (VSS), U3.G5 (VSS), U3.H10 (VSS), U3.J5 (VSS), U3.K8 (VSS), U3.N2 (VSS), U3.N5 (VSS), U3.P4 (VSS), U3.P6 (VSS), C123.2, C124.2, C125.2, C126.2, C127.2, C128.2, C129.2, C130.2, C131.2, C132.2
- net eMMC_D3: now reaches U3.B2 (DAT3)
- net eMMC_D4: now reaches U3.B3 (DAT4)
- net eMMC_D5: now reaches U3.B4 (DAT5)
- net eMMC_D6: now reaches U3.B5 (DAT6)
- net eMMC_D7: now reaches U3.B6 (DAT7)
- net at U3.C2 (VDDI): now also C123.1
- net VCCIO_FLASH: now reaches U3.C6 (VDD)
- net VCCIO_FLASH: now also U3.M4 (VDD), U3.N4 (VDD), U3.P3 (VDD), U3.P5 (VDD), C126.1, C127.1, C129.1, C131.1, C132.1, R67.2, R69.2
- net VCC_3V3: now reaches U3.E6 (VDDF)
- net VCC_3V3: now also U3.F5 (VDDF), U3.J10 (VDDF), U3.K9 (VDDF), C124.1, C125.1, C130.1, R68.2
- net eMMC_DATA_STROBE: now reaches U3.H5 (DATASTROBE)
- net eMMC_RSTn: now reaches U3.K5 (RSTN)
- net eMMC_RSTn: now also C128.1, R68.1
- net eMMC_CMD: now reaches U3.M5 (CDM)
- net eMMC_CMD: now also R69.1
- net eMMC_CLKOUT: now reaches U3.M6 (CLK)
- no-connect marks 0 -> 120

Commit message: MIPI IS FAKE
Parts:
- added C133: 100nF X5R 10V, Capacitor_SMD:C_0402_1005Metric, symbol Device:C
- added C134: 10uF X5R 10V, Capacitor_SMD:C_0603_1608Metric, symbol Device:C
- added Card1: TF PUSH, lcsc:TF-SMD_TF-PUSH, symbol lcsc:TFPUSH
- added R70, R71, R72, R73, R74, R75: 22R 5%, Resistor_SMD:R_0402_1005Metric, symbol Device:R
- added U19, U20, U21, U22, U23, U24, U25: ESD5311X, lcsc:DFN1006-2L-BI, symbol lcsc:ESD5311X_C2844730
Connections:
- net GND: now also C133.2, C134.2, Card1.10, Card1.11, Card1.12, Card1.13, Card1.6 (VSS), U19.1, U20.1, U21.1, U22.1, U23.1, U24.1, U25.1
- net VCCIO_FLASH: now also R68.2
- net VCC_3V3: no longer R68.2
- new net: Card1.7 (DAT0), R73.2, U21.2
- new net: Card1.3 (CMD), R72.2, U23.2
- new net: Card1.1 (DAT2), R70.2, U25.2
- new net: Card1.8 (DAT1), R74.2, U20.2
- new net: Card1.2 (CD/DAT3), R71.2, U24.2
- new net: Card1.9 (CD), R75.2, U19.2
- new net SDMMC0_CLK: Card1.5 (CLX), U22.2
- new net SDMMC0_CMD: R72.1
- new net SDMMC0_D0: R73.1
- new net SDMMC0_D1: R74.1
- new net SDMMC0_D2/ARMJTAG_TCK: R70.1
- new net SDMMC0_D3/ARMJTAG_TMS: R71.1
- new net SDMMC0_DET_L: R75.1
- new net VCC3V3_SD: C133.1, C134.1, Card1.4 (VDD)
Other:
- note added: "Close to microSD Card"
- moved on the sheet: C129, R69, U2

Commit message: add in pcie and ddr4
Parts:
- added C200, C222: 22uF X5R 6.3V, Capacitor_SMD:C_0603_1608Metric, symbol Device:C
- added C201, C202, C223, C224, C243, C244, C278: 10uF X5R 6.3V, Capacitor_SMD:C_0603_1608Metric, symbol Device:C
- added C203, C225: 1uF X5R 10V, Capacitor_SMD:C_0402_1005Metric, symbol Device:C
- added C204, C205, C206, C207, C208, C209, C210, C211, C212, C213, C214, C215, C216, C217, C218, C219, C220, C221, C226, C227, C228, C229, C230, C231, C232, C233, C234, C235, C236, C237, C238, C239, C240, C241, C245, C246, C247, C248, C250, C251: 100nF X5R 10V, Capacitor_SMD:C_0402_1005Metric, symbol Device:C
- added C242: 10uF X5R 10V, Capacitor_SMD:C_0603_1608Metric, symbol Device:C
- added C249, C275, C276, C277, C280, C281: 4.7uF X5R 6.3V, Capacitor_SMD:C_0402_1005Metric, symbol Device:C
- added C274, C279, C282, C283: 100nF X5R 10V, Capacitor_SMD:C_0201_0603Metric, symbol Device:C
- added R142, R143: 240R 5%, Resistor_SMD:R_0402_1005Metric, symbol Device:R
- added R144: 0R 5%, Resistor_SMD:R_0201_0603Metric, symbol Device:R
- added R150: 120R 1%, Resistor_SMD:R_0201_0603Metric, symbol Device:R
- added unit 4 of U1
Connections:
- net GND: now also U2.A10 (VSS), U2.A3 (VSS), U2.AB10 (VSS), U2.AB3 (VSS), U2.AB5 (VSS), U2.AB8 (VSS), U2.C1 (VSS), U2.C12 (VSS), U2.C5 (VSS), U2.C8 (VSS), U2.D11 (VSS), U2.D2 (VSS), U2.D4 (VSS), U2.D9 (VSS), U2.E1 (VSS), U2.E12 (VSS), U2.E5 (VSS), U2.E8 (VSS), U2.G1 (VSS), U2.G10 (VSS), U2.G12 (VSS), U2.G3 (VSS), U2.G5 (VSS), U2.G8 (VSS), U2.J1 (VSS), U2.J10 (VSS), U2.J12 (VSS), U2.J3 (VSS), U2.K11 (VSS), U2.K2 (VSS), U2.K4 (VSS), U2.K9 (VSS), U2.N11 (VSS), U2.N2 (VSS), U2.N4 (VSS), U2.N9 (VSS), U2.P1 (VSS), U2.P10 (VSS), U2.P12 (VSS), U2.P3 (VSS), U2.T1 (VSS), U2.T10 (VSS), U2.T12 (VSS), U2.T3 (VSS), U2.T5 (VSS), U2.T8 (VSS), U2.V1 (VSS), U2.V12 (VSS), U2.V5 (VSS), U2.V8 (VSS), U2.W11 (VSS), U2.W2 (VSS), U2.W4 (VSS), U2.W9 (VSS), U2.Y1 (VSS), U2.Y12 (VSS), U2.Y5 (VSS), U2.Y8 (VSS), C200.2, C201.2, C202.2, C203.2, C204.2, C205.2, C206.2, C207.2, C208.2, C209.2, C210.2, C211.2, C212.2, C213.2, C214.2, C215.2, C216.2, C217.2, C218.2, C219.2, C220.2, C221.2, C222.2, C223.2, C224.2, C225.2, C226.2, C227.2, C228.2, C229.2, C230.2, C231.2, C232.2, C233.2, C234.2, C235.2, C236.2, C237.2, C238.2, C239.2, C240.2, C241.2, C242.2, C243.2, C244.2, C245.2, C246.2, C247.2, C248.2, C249.2, C250.2, C251.2, C274.2, C275.2, C276.2, C277.2, C278.2, C279.2, C280.2, C281.2, C282.2, C283.2, U1.J8 (DDR_AVSS)
- net DDRPHY_VDDQ: now reaches U2.A4 (VDD2)
- net DDRPHY_VDDQ: now also U2.A9 (VDD2), U2.AB4 (VDD2), U2.AB9 (VDD2), U2.F5 (VDD2), U2.F8 (VDD2), U2.H1 (VDD2), U2.H12 (VDD2), U2.H5 (VDD2), U2.H8 (VDD2), U2.K1 (VDD2), U2.K10 (VDD2), U2.K12 (VDD2), U2.K3 (VDD2), U2.N1 (VDD2), U2.N10 (VDD2), U2.N12 (VDD2), U2.N3 (VDD2), U2.R1 (VDD2), U2.R12 (VDD2), U2.R5 (VDD2), U2.R8 (VDD2), U2.U5 (VDD2), U2.U8 (VDD2), C200.1, C201.1, C202.1, C203.1, C204.1, C205.1, C206.1, C207.1, C208.1, C209.1, C210.1, C211.1, C212.1, C213.1, C214.1, C215.1, C216.1, C217.1, C218.1, C219.1, C220.1, C221.1, C274.1, C275.1, C278.1, C279.1, C280.1, R150.2, U1.H11 (DDRPHY_VDDQ), U1.H12 (DDRPHY_VDDQ), U1.H14 (DDRPHY_VDDQ), U1.H15 (DDRPHY_VDDQ), U1.H9 (DDRPHY_VDDQ), U1.J9 (DDRPHY_VDDQ), U1.L9 (DDRPHY_VDDQ), U1.M9 (DDRPHY_VDDQ)
- net at U2.A5 (ZQ0): now also R143.1
- net at U2.A8 (ZQ1): now also R142.1
- net DDRPHY_VDDQL: now reaches U2.AA10 (VDDQ)
- net DDRPHY_VDDQL: now also U2.AA3 (VDDQ), U2.AA5 (VDDQ), U2.AA8 (VDDQ), U2.B10 (VDDQ), U2.B3 (VDDQ), U2.B5 (VDDQ), U2.B8 (VDDQ), U2.D1 (VDDQ), U2.D12 (VDDQ), U2.D5 (VDDQ), U2.D8 (VDDQ), U2.F10 (VDDQ), U2.F3 (VDDQ), U2.U10 (VDDQ), U2.U3 (VDDQ), U2.W1 (VDDQ), U2.W12 (VDDQ), U2.W5 (VDDQ), U2.W8 (VDDQ), C222.1, C223.1, C224.1, C225.1, C226.1, C227.1, C228.1, C229.1, C230.1, C231.1, C232.1, C233.1, C234.1, C235.1, C236.1, C237.1, C238.1, C239.1, C240.1, C241.1, C242.1, C276.1, C277.1, C281.1, C282.1, C283.1, R142.2, R143.2, U1.J11 (DDRPHY_VDDQL), U1.J12 (DDRPHY_VDDQL), U1.J14 (DDRPHY_VDDQL), U1.K10 (DDRPHY_VDDQL), U1.L10 (DDRPHY_VDDQL), U1.M10 (DDRPHY_VDDQL)
- net LPDDR4_DQ8_B: now reaches U2.AA11 (DQ8_b)
- net LPDDR4_DQ8_B: now also U1.A16 (DDR_DQ8_B)
- net LPDDR4_DQ0_B: now reaches U2.AA2 (DQ0_b)
- net LPDDR4_DQ0_B: now also U1.B10 (DDR_DQ0_B)
- net LPDDR4_DQ7_B: now reaches U2.AA4 (DQ7_b)
- net LPDDR4_DQ7_B: now also U1.E14 (DDR_DQ7_B)
- net LPDDR4_DQ15_B: now reaches U2.AA9 (DQ15_b)
- net LPDDR4_DQ15_B: now also U1.B14 (DDR_DQ15_B)
- net LPDDR4_DQ8_A: now reaches U2.B11 (DQ8_a)
- net LPDDR4_DQ8_A: now also U1.M1 (DDR_DQ8_A)
- net LPDDR4_DQ0_A: now reaches U2.B2 (DQ0_a)
- net LPDDR4_DQ0_A: now also U1.F2 (DDR_DQ0_A)
- net LPDDR4_DQ7_A: now reaches U2.B4 (DQ7_a)
- net LPDDR4_DQ7_A: now also U1.H4 (DDR_DQ7_A)
- net LPDDR4_DQ15_A: now reaches U2.B9 (DQ15_a)
- net LPDDR4_DQ15_A: now also U1.L4 (DDR_DQ15_A)
- net LPDDR4_DM1_A: now reaches U2.C10 (DMI1_a)
- net LPDDR4_DM1_A: now also U1.J4 (DDR_DM1_A)
- net LPDDR4_DQ9_A: now reaches U2.C11 (DQ9_a)
- net LPDDR4_DQ9_A: now also U1.N2 (DDR_DQ9_A)
- net LPDDR4_DQ1_A: now reaches U2.C2 (DQ1_a)
- net LPDDR4_DQ1_A: now also U1.E1 (DDR_DQ1_A)
- net LPDDR4_DM0_A: now reaches U2.C3 (DMI0_a)
- net LPDDR4_DM0_A: now also U1.H5 (DDR_DM0_A)
- net LPDDR4_DQ6_A: now reaches U2.C4 (DQ6_a)
- net LPDDR4_DQ6_A: now also U1.H1 (DDR_DQ6_A)
- net LPDDR4_DQ14_A: now reaches U2.C9 (DQ14_a)
- net LPDDR4_DQ14_A: now also U1.J7 (DDR_DQ14_A)
- net LPDDR4_DQS1P_A: now reaches U2.D10 (DQS1_t_a)
- net LPDDR4_DQS1P_A: now also U1.L2 (DDR_DQS1P_A)
- net LPDDR4_DQS0P_A: now reaches U2.D3 (DQS0_t_a)
- net LPDDR4_DQS0P_A: now also U1.G1 (DDR_DQS0P_A)
- net LPDDR4_DQS1N_A: now reaches U2.E10 (DQS1_c_a)
- net LPDDR4_DQS1N_A: now also U1.L1 (DDR_DQS1N_A)
- net LPDDR4_DQ10_A: now reaches U2.E11 (DQ10_a)
- net LPDDR4_DQ10_A: now also U1.L7 (DDR_DQ10_A)
- net LPDDR4_DQ2_A: now reaches U2.E2 (DQ2_a)
- net LPDDR4_DQ2_A: now also U1.E2 (DDR_DQ2_A)
- net LPDDR4_DQS0N_A: now reaches U2.E3 (DQS0_c_a)
- net LPDDR4_DQS0N_A: now also U1.G2 (DDR_DQS0N_A)
- net LPDDR4_DQ5_A: now reaches U2.E4 (DQ5_a)
- net LPDDR4_DQ5_A: now also U1.J2 (DDR_DQ5_A)
- net LPDDR4_DQ13_A: now reaches U2.E9 (DQ13_a)
- net LPDDR4_DQ13_A: now also U1.J6 (DDR_DQ13_A)
- net VCC1V8_DDR: now reaches U2.F1 (VDD1)
- net VCC1V8_DDR: now also U2.F12 (VDD1), U2.G4 (VDD1), U2.G9 (VDD1), U2.T4 (VDD1), U2.T9 (VDD1), U2.U1 (VDD1), U2.U12 (VDD1), C243.1, C244.1, C245.1, C246.1, C247.1, C248.1, C249.1, C250.1, C251.1, R144.2
- net LPDDR4_DQ11_A: now reaches U2.F11 (DQ11_a)
- net LPDDR4_DQ11_A: now also U1.L6 (DDR_DQ11_A)
- net LPDDR4_DQ3_A: now reaches U2.F2 (DQ3_a)
- net LPDDR4_DQ3_A: now also U1.D1 (DDR_DQ3_A)
- net LPDDR4_DQ4_A: now reaches U2.F4 (DQ4_a)
- net LPDDR4_DQ4_A: now also U1.J1 (DDR_DQ4_A)
- net LPDDR4_DQ12_A: now reaches U2.F9 (DQ12_a)
- net LPDDR4_DQ12_A: now also U1.K2 (DDR_DQ12_A)
- net LPDDR4_ODT0_CA_A: now reaches U2.G2 (ODT_CA_a1)/2))
- net LPDDR4_ODT0_CA_A: now also U1.C1 (AC8)
- net LPDDR4_A3_A: now reaches U2.H10 (CA3_a)
- net LPDDR4_A3_A: now also U1.C4 (AC12)
- net LPDDR4_A4_A: now reaches U2.H11 (CA4_a)
- net LPDDR4_A4_A: now also U1.C5 (AC14)
- net LPDDR4_A0_A: now reaches U2.H2 (CA0_a)
- net LPDDR4_A0_A: now also U1.C2 (AC11)
- net LPDDR4_CS1n_A: now reaches U2.H3 (CS1_a)
- net LPDDR4_CS1n_A: now also U1.B2 (AC26)
- net LPDDR4_CS0n_A: now reaches U2.H4 (CS0_a)
- net LPDDR4_CS0n_A: now also U1.A2 (AC25)
- net LPDDR4_A2_A: now reaches U2.H9 (CA2_a)
- net LPDDR4_A2_A: now also U1.E4 (AC15)
- net LPDDR4_A5_A: now reaches U2.J11 (CA5_a)
- net LPDDR4_A5_A: now also U1.D5 (AC16)
- net LPDDR4_A1_A: now reaches U2.J2 (CA1_a)
- net LPDDR4_A1_A: now also U1.B1 (AC2)
- net LPDDR4_CKE0_A: now reaches U2.J4 (CKE0_a)
- net LPDDR4_CKE0_A: now also U1.B3 (AC22)
- net LPDDR4_CKE1_A: now reaches U2.J5 (CKE1_a)
- net LPDDR4_CKE1_A: now also U1.F4 (AC3)
- net LPDDR4_CLKP_A: now reaches U2.J8 (CK_t_a)
- net LPDDR4_CLKP_A: now also U1.B4 (AC23)
- net LPDDR4_CLKN_A: now reaches U2.J9 (CK_c_a)
- net LPDDR4_CLKN_A: now also U1.A4 (AC24)
- net LPDDR4_A5_B: now reaches U2.P11 (CA5_b)
- net LPDDR4_A5_B: now also U1.B7 (AC5)
- net LPDDR4_A1_B: now reaches U2.P2 (CA1_b)
- net LPDDR4_A1_B: now also U1.A7 (AC6)
- net LPDDR4_CKE0_B: now reaches U2.P4 (CKE0_b)
- net LPDDR4_CKE0_B: now also U1.D6 (AC10)
- net LPDDR4_CKE1_B: now reaches U2.P5 (CKE1_b)
- net LPDDR4_CKE1_B: now also U1.E6 (AC17)
- net LPDDR4_CLKP_B: now reaches U2.P8 (CK_t_b)
- net LPDDR4_CLKP_B: now also U1.B6 (AC0)
- net LPDDR4_CLKN_B: now reaches U2.P9 (CK_c_b)
- net LPDDR4_CLKN_B: now also U1.A5 (AC9)
- net LPDDR4_A3_B: now reaches U2.R10 (CA3_b)
- net LPDDR4_A3_B: now also U1.D9 (AC4)
- net LPDDR4_A4_B: now reaches U2.R11 (CA4_b)
- net LPDDR4_A4_B: now also U1.E9 (AC19)
- net LPDDR4_A0_B: now reaches U2.R2 (CA0_b)
- net LPDDR4_A0_B: now also U1.B8 (AC13)
- net LPDDR4_CS1n_B: now reaches U2.R3 (CS1_b)
- net LPDDR4_CS1n_B: now also U1.E8 (AC27)
- net LPDDR4_CS0n_B: now reaches U2.R4 (CS0_b)
- net LPDDR4_CS0n_B: now also U1.D8 (AC28)
- net LPDDR4_A2_B: now reaches U2.R9 (CA2_b)
- net LPDDR4_A2_B: now also U1.E11 (AC18)
- net LPDDR4_RESETn: now reaches U2.T11 (RESET_n)
- net LPDDR4_RESETn: now also U1.F11 (AC29)
- net LPDDR4_ODT0_CA_B: now reaches U2.T2 (ODT_CA_b1)/2))
- net LPDDR4_ODT0_CA_B: now also U1.A8 (AC7)
- net LPDDR4_DQ11_B: now reaches U2.U11 (DQ11_b)
- net LPDDR4_DQ11_B: now also U1.B18 (DDR_DQ11_B)
- net LPDDR4_DQ3_B: now reaches U2.U2 (DQ3_b)
- net LPDDR4_DQ3_B: now also U1.E12 (DDR_DQ3_B)
- net LPDDR4_DQ4_B: now reaches U2.U4 (DQ4_b)
- net LPDDR4_DQ4_B: now also U1.A12 (DDR_DQ4_B)
- net LPDDR4_DQ12_B: now reaches U2.U9 (DQ12_b)
- net LPDDR4_DQ12_B: now also U1.B13 (DDR_DQ12_B)
- net LPDDR4_DQS1N_B: now reaches U2.V10 (DQS1_c_b)
- net LPDDR4_DQS1N_B: now also U1.A15 (DDR_DQS1N_B)
- net LPDDR4_DQ10_B: now reaches U2.V11 (DQ10_b)
- net LPDDR4_DQ10_B: now also U1.A17 (DDR_DQ10_B)
- net LPDDR4_DQ2_B: now reaches U2.V2 (DQ2_b)
- net LPDDR4_DQ2_B: now also U1.D12 (DDR_DQ2_B)
- net LPDDR4_DQS0N_B: now reaches U2.V3 (DQS0_c_b)
- net LPDDR4_DQS0N_B: now also U1.B11 (DDR_DQS0N_B)
- net LPDDR4_DQ5_B: now reaches U2.V4 (DQ5_b)
- net LPDDR4_DQ5_B: now also U1.D15 (DDR_DQ5_B)
- net LPDDR4_DQ13_B: now reaches U2.V9 (DQ13_b)
- net LPDDR4_DQ13_B: now also U1.A13 (DDR_DQ13_B)
- net LPDDR4_DQS1P_B: now reaches U2.W10 (DQS1_t_b)
- net LPDDR4_DQS1P_B: now also U1.B15 (DDR_DQS1P_B)
- net LPDDR4_DQS0P_B: now reaches U2.W3 (DQS0_t_b)
- net LPDDR4_DQS0P_B: now also U1.A11 (DDR_DQS0P_B)
- net LPDDR4_DM1_B: now reaches U2.Y10 (DMI1_b)
- net LPDDR4_DM1_B: now also U1.E17 (DDR_DM1_B)
- net LPDDR4_DQ9_B: now reaches U2.Y11 (DQ9_b)
- net LPDDR4_DQ9_B: now also U1.B17 (DDR_DQ9_B)
- net LPDDR4_DQ1_B: now reaches U2.Y2 (DQ1_b)
- net LPDDR4_DQ1_B: now also U1.A9 (DDR_DQ1_B)
- net LPDDR4_DM0_B: now reaches U2.Y3 (DMI0_b)
- net LPDDR4_DM0_B: now also U1.D14 (DDR_DM0_B)
- net LPDDR4_DQ6_B: now reaches U2.Y4 (DQ6_b)
- net LPDDR4_DQ6_B: now also U1.E15 (DDR_DQ6_B)
- net LPDDR4_DQ14_B: now reaches U2.Y9 (DQ14_b)
- net LPDDR4_DQ14_B: now also U1.D17 (DDR_DQ14_B)
- net LPDDR4_ODT1_CA_A: now reaches U1.F7 (AC21)
- net LPDDR4_ODT1_CA_B: now reaches U1.F8 (AC20)
- net at U1.H7 (DDR_RZQ): now also R150.1
- new net VCCA1V8_PMU: R144.1
- no-connect marks 120 -> 150
Other:
- note added: "Caps should be placed under RK3568"
- note added: "For LPDDR4/LPDDR4x mode, a 120 ohm +/-1% tolerance external resistor must be connected between the DDR_RZQ pin and DDRPHY_VDDQ pi"
- moved on the sheet: C123, C124, C125, C126, C127, C128, C129, C130, C131, C132, C133, C134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

Commit message: finished schematic!
Parts:
- added C337, C338: 100nF X5R 10V, Capacitor_SMD:C_0201_0603Metric, symbol Device:C
- added R195, R196: 22R 5%, Resistor_SMD:R_0402_1005Metric, symbol Device:R
- added TP5, TP6, TP7, TP8, TP9: TestPoint, TestPoint:TestPoint_Pad_D1.0mm, symbol Connector:TestPoint
- added unit 9 of U1
- added unit 8 of U1
Connections:
- net GND: now also C337.2, C338.2, TP6.1, TP8.1
- net SDMMC0_CLK: now also R196.2
- net SDMMC0_CMD: now also U1.H27 (GPIO2_A1_U)
- net SDMMC0_D0: now also U1.J25 (GPIO1_D5_U)
- net SDMMC0_D1: now also U1.J24 (GPIO1_D6_U)
- net SDMMC0_D2/ARMJTAG_TCK: now also TP9.1, U1.H26 (GPIO1_D7_U)
- net SDMMC0_D3/ARMJTAG_TMS: now also TP7.1, U1.J23 (GPIO2_A0_U)
- net VCCIO_FLASH: now also C337.1, U1.H18 (VCCIO2)
- net eMMC_CLKOUT: now also R195.1
- net eMMC_CMD: now also U1.B22 (GPIO1_C4_U)
- net eMMC_D0: now also TP5.1, U1.A24 (GPIO1_B4_U)
- net eMMC_D1: now also U1.C21 (GPIO1_B5_U)
- net eMMC_D2: now also U1.B24 (GPIO1_B6_U)
- net eMMC_D3: now also U1.D21 (GPIO1_B7_U)
- net eMMC_D4: now also U1.A25 (GPIO1_C0_U)
- net eMMC_D5: now also U1.E21 (GPIO1_C1_U)
- net eMMC_D6: now also U1.E22 (GPIO1_C2_U)
- net eMMC_D7: now also U1.B25 (GPIO1_C3_U)
- net eMMC_DATA_STROBE: now also U1.A26 (GPIO1_C6_D)
- net eMMC_RSTn: now also U1.F20 (GPIO1_C7_D)
- new net: R196.1, U1.H28 (GPIO2_A2_D)
- new net: R195.2, U1.A23 (GPIO1_C5_D)
- new net VCCIO_SD: C338.1, U1.L22 (VCCIO3)
- no-connect marks 150 -> 156
Other:
- note added: "32 GB eMMC"
- note added: "8GB LPDDR4 RAM"
- note added: "For eMMC or Nand Flash: If eMMC_D0/FLASH_D0=0V at after power on and reset, then system will enter into Maskrom mode."
- note added: "MicroSD Card"
- note added: "Reserved for ARM JTAG debug"
- note added: "Test point must be placed on the line, and no branch can be added"
- moved on the sheet: R150, U1E

Commit message: finished beautifying schematic
Connections:
- no-connect marks 156 -> 155
Other:
- note added: "Decoupling"
- note added: "Frost"
- note added: "LPDDR4 Ram"
- note added: "RK3568"
- note added: "eMMC"
- note removed: "32 GB eMMC"
- note removed: "8GB LPDDR4 RAM"
- moved on the sheet: C123, C124, C125, C126, C127, C128, C129, C130, C131, C132, C133, C134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
