File: hardware/board/ethernet.kicad_sch (KiCad schematic)
At the start: 0 parts

Commit message: start of ethernet
Parts:
- added C177, C178: 20pF C0G 50V, Capacitor_SMD:C_0402_1005Metric, symbol Device:C
- added C179, C180, C182, C183, C184, C185, C187, C190, C191, C193: 100nF X5R 10V, Capacitor_SMD:C_0402_1005Metric, symbol Device:C
- added C181, C186, C189, C192: 4.7uF X5R 10V, Capacitor_SMD:C_0603_1608Metric, symbol Device:C
- added C188: 1uF X5R 10V, Capacitor_SMD:C_0402_1005Metric, symbol Device:C
- added D17: LED GREEN, LED_SMD:LED_0603_1608Metric, symbol Device:LED
- added D18: LED YELLOW, LED_SMD:LED_0603_1608Metric, symbol Device:LED
- added R100: 120R 5%, Resistor_SMD:R_0402_1005Metric, symbol Device:R
- added R101: 100R 5%, Resistor_SMD:R_0402_1005Metric, symbol Device:R
- added R102: 2.49K 1%, Resistor_SMD:R_0402_1005Metric, symbol Device:R
- added R103, R104, R128, R130, R131: 0R 5%, Resistor_SMD:R_0402_1005Metric, symbol Device:R
- added R105: 1.8K 5%, Resistor_SMD:R_0402_1005Metric, symbol Device:R
- added R106, R107, R108, R109, R110, R111: 22R 5%, Resistor_SMD:R_0402_1005Metric, symbol Device:R
- added R112, R113, R114, R115, R116, R117, R118, R119, R120, R121, R122, R123, R124, R125, R126: 4.7K 5%, Resistor_SMD:R_0402_1005Metric, symbol Device:R
- added R127, R129: 510R 5%, Resistor_SMD:R_0402_1005Metric, symbol Device:R
- added RJ5: 2-406549-1, lcsc:RJ45-TH_2-406549-1, symbol lcsc:2-406549-1
- added U36: RTL8211F-CG, lcsc:WQFN-40_L5.0-W5.0-P0.4-BL-EP, symbol lcsc:RTL8211F-CG
- added U37: TFM252012ALVA2R2MTAA, lcsc:L1008, symbol lcsc:TFM252012ALVA2R2MTAA
- added U38: QG2439S, lcsc:SMD-24_L15.1-W7.1-P1.00-LS10.0-BL, symbol lcsc:QG2439S
- added X4: X322525MOB4SI, lcsc:CRYSTAL-SMD_4P-L3.2-W2.5-BL, symbol lcsc:X322525MOB4SI
Connections:
- new net: C179.1, R104.2, U36.12 (PHYRSTB)
- new net: R103.1, U36.31 (INTB/PMEB)
- new net: D18.2 (A), R127.2
- new net: D17.1 (K), R129.1
- new net: D18.1 (K), R128.2
- new net GMAC0_MCLKINOUT: R100.2, R101.1, R104.1
- new net GMAC0_MDC: U36.13 (MDC)
- new net GMAC0_MDIO: R105.1, U36.14 (MDIO)
- new net GMAC0_RXCLK: R110.1
- new net GMAC0_RXD0: R106.1
- new net GMAC0_RXD1: R107.1
- new net GMAC0_RXD2: R108.1
- new net GMAC0_RXD3: R109.1
- new net GMAC0_RXDV_CRS: R111.1
- new net GMAC0_TXCLK: U36.20 (TXC)
- new net GMAC0_TXD0: U36.18 (TXD0)
- new net GMAC0_TXD1: U36.17 (TXD1)
- new net GMAC0_TXD2: U36.16 (TXD2)
- new net GMAC0_TXD3: U36.15 (TXD3)
- new net GMAC0_TXEN: U36.19 (TXCTL)
- new net GND: C177.2, C178.2, C179.2, C180.2, C181.2, C182.2, C183.2, C184.2, C185.2, C186.2, C187.2, C188.2, C189.2, C190.2, C191.2, C192.2, C193.2, R100.1, R102.2, R112.2, R114.2, R116.2, R117.2, R119.2, R120.2, R121.2, R123.2, R125.2, R129.2, U36.41 (GND), X4.2 (GND), X4.4 (GND)
- new net PHY0_CLKOUT125: R101.2, U36.35 (CLKOUT)
- new net PHY0_LED0/CFG_EXT: R103.2, R112.1, R113.2, U36.32 (CFG_EXT/LED0)
- new net PHY0_LED1/CFG_LDO0: R116.1, U36.33 (CFG_LDO0/LED1)
- new net PHY0_LED2/CFG_LDO1: D17.2 (A), R114.1, R115.2, R128.1, U36.34 (CFG_LDO1/LED2)
- new net PHY0_MDI0+: U36.1 (MDIP0)
- new net PHY0_MDI0-: U36.2 (MDIN0)
- new net PHY0_MDI1+: U36.4 (MDIP1)
- new net PHY0_MDI1-: U36.5 (MDIN1)
- new net PHY0_MDI2+: U36.6 (MDIP2)
- new net PHY0_MDI2-: U36.7 (MDIN2)
- new net PHY0_MDI3+: U36.9 (MDIP3)
- new net PHY0_MDI3-: U36.10 (MDIN3)
- new net PHY0_REG_OUT: U36.30 (REG_OUT/LDO_OUT), U37.2
- new net PHY0_RXCLK/PHYAD1: R110.2, R119.1, U36.27 (PHYAD1/RXC)
- new net PHY0_RXD0/RXDLY: R106.2, R121.1, R122.2, U36.25 (RXDLY/RXD0)
- new net PHY0_RXD1/TXDLY: R107.2, R123.1, R124.2, U36.24 (TXDLY/RXD1)
- new net PHY0_RXD2/PLLOFF: R108.2, R125.1, R126.2, U36.23 (PLLOFF/RXD2)
- new net PHY0_RXD3/PHYAD0: R109.2, R117.1, R118.2, U36.22 (PHYAD0/RXD3)
- new net PHY0_RXDV/PHYAD2: R111.2, R120.1, U36.26 (PHYAD2/RXCTL)
- new net PHY0_XTALIN: C178.1, U36.36 (XTAL_IN), X4.3 (OSC2)
- new net PHY0_XTALOUT: C177.1, U36.37 (XTAL_OUT/EXT_CLK), X4.1 (OSC1)
- new net RSET0: R102.1, U36.39 (RSET)
- new net VCC3V3_PHY0: C189.1, C190.1, C191.1, C192.1, C193.1, R113.1, R115.1, R127.1, R130.2, U36.11 (AVDD33), U36.29 (DVDD33), U36.40 (AVDD33)
- new net VCCIO_PHY0: C186.1, C187.1, C188.1, R105.2, R118.1, R122.1, R124.1, R126.1, U36.28 (DVDD_RG)
- new net VCC_3V3: R130.1
- new net VDD10_PHY0: C180.1, C181.1, C182.1, C183.1, C184.1, C185.1, U36.21 (DVDD10), U36.3 (AVDD10), U36.38 (AVDD10), U36.8 (AVDD10), U37.1
Other:
- note added: "Close to PHY"
- note added: "Close to PIN11,40"
- note added: "Close to PIN21"
- note added: "Close to PIN28"
- note added: "Close to PIN29"
- note added: "Close to PIN3,8,38"
- note added: "Close to PIN30"
- note added: "PHY Address Config"
- note added: "Pull-up for additional 2ns delay to RXC for data latching"
- note added: "Pull-up for additional 2ns delay to TXC for data latching"
- note added: "Pull-up to disable PLL @ ALDPS mode(Low power mode)"
- note added: "VCC_PHY0_IO Voltage Config"

Commit message: finish ethernet
Parts:
- removed D17: LED GREEN, LED_SMD:LED_0603_1608Metric, symbol Device:LED
- removed D18: LED YELLOW, LED_SMD:LED_0603_1608Metric, symbol Device:LED
- removed R129: 510R 5%, Resistor_SMD:R_0402_1005Metric, symbol Device:R
- removed RJ5: 2-406549-1, lcsc:RJ45-TH_2-406549-1, symbol lcsc:2-406549-1
- removed U38: QG2439S, lcsc:SMD-24_L15.1-W7.1-P1.00-LS10.0-BL, symbol lcsc:QG2439S
- added C194, C195, C196, C197: 10nF X5R 25V, Capacitor_SMD:C_0402_1005Metric, symbol Device:C
- added FB11: 120@100MHz 25% 2A, Inductor_SMD:L_0603_1608Metric, symbol Device:FerriteBead
- added R132, R133, R134, R135, R136, R137, R138: 0R 5%, Resistor_SMD:R_0402_1005Metric, symbol Device:R
- added RJ1: HY911130A, lcsc:RJ45-TH_10P-P2.54-S2.54_L16.1-W21.4_HY911130A, symbol lcsc:HY911130A
- added U38, U39, U40, U41, U42, U43, U44, U45: ESD5451N_C5261080, lcsc:DFN1006-2L-BI, symbol lcsc:ESD5451N_C5261080
- R128: value 0R 5% -> 510R 5%
Connections:
- net GND: now also C194.2, C195.2, C196.2, C197.2, FB11.2, RJ1.12, RJ1.2 (10), U38.1, U39.1, U40.1, U41.1, U42.1, U43.1, U44.1, U45.1
- net PHY0_LED1/CFG_LDO0: now also R127.2
- net PHY0_LED2/CFG_LDO1: now also R128.2; no longer R128.1
- net PHY0_MDI0+: now also R131.1
- net PHY0_MDI0-: now also R132.1
- net PHY0_MDI1+: now also R133.1
- net PHY0_MDI1-: now also R134.1
- net PHY0_MDI2+: now also R135.1
- net PHY0_MDI2-: now also R136.1
- net PHY0_MDI3+: now also R137.1
- net PHY0_MDI3-: now also R138.1
- net VCC3V3_PHY0: now also RJ1.14; no longer R127.1
- net at R131.2: now also RJ1.2 (10), U38.2
- new net: R132.2, RJ1.3, U39.2
- new net: C194.1, C195.1, C196.1, C197.1, RJ1.1 (9)
- new net: R138.2, RJ1.1 (9), U45.2
- new net: R136.2, RJ1.7, U43.2
- new net: R134.2, RJ1.5, U41.2
- new net: FB11.1, RJ1.15 (SH), RJ1.16 (SH)
- new net: R133.2, RJ1.4, U40.2
- new net: R135.2, RJ1.6, U42.2
- new net: R137.2, RJ1.8, U44.2
- new net PHY0_LED1_N: R127.1, RJ1.11
- new net PHY0_LED2_N: R128.1, RJ1.13
Other:
- note added: "Green"
- note added: "Might replace with ESD5344D"
- note added: "Yellow"
- moved on the sheet: R127, R131

Commit message: aaa
Connections:
- net GMAC0_MCLKINOUT: no longer R104.1
- net PHY0_LED0/CFG_EXT: no longer R103.2
- net PHY0_LED1_N renamed PHY0_LED1_P
- new net GMAC0_INT/PMEB_GPIO3_C0: R103.2
- new net GMAC0_RSTn_GPIO3_B0: R104.1
Other:
- note added: "Might be optional"
Changed lines of the file:
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@@
+		)
+	)
+	(text "Might be optional"
+		(exclude_from_sim no)
+		(at 200.66 74.93 0)
+		(effects
+			(font
+				(size 1.27 1.27)
+			)
 		)
 	)
@@
 		)
 	)
-	(label "PHY0_LED1_N"
+	(label "PHY0_LED1_P"
 		(at 356.87 100.33 180)
 		(effects
@@
 		)
 	)
-	(label "PHY0_LED1_N"
+	(label "PHY0_LED1_P"
 		(at 369.57 144.78 180)
 		(effects
@@
 		)
 	)
-	(global_label "PHY0_LED0{slash}CFG_EXT"
+	(global_label "GMAC0_INT{slash}PMEB_GPIO3_C0"
 		(shape output)
 		(at 173.99 114.3 0)
@@
 		)
 		(property "Intersheetrefs" "${INTERSHEET_REFS}"
-			(at 196.7508 114.3 0)
+			(at 203.7056 114.3 0)
 			(effects
 				(font
@@
 		)
 	)
-	(global_label "GMAC0_MCLKINOUT"
+	(global_label "GMAC0_RSTn_GPIO3_B0"
 		(shape input)
 		(at 33.02 119.38 180)
@@
 		)
 		(property "Intersheetrefs" "${INTERSHEET_REFS}"
-			(at 12.1943 119.38 0)
+			(at 8.0821 119.38 0)
 			(effects
 				(font

Commit message: finished schematic!
Parts:
- added C362: 100nF X5R 10V, Capacitor_SMD:C_0201_0603Metric, symbol Device:C
- added C363: 1uF X5R 6.3V, Capacitor_SMD:C_0402_1005Metric, symbol Device:C
- added R200, R201: 2.2K 5%, Resistor_SMD:R_0402_1005Metric, symbol Device:R
- added R202, R203, R204, R205, R206, R207: 22R 5%, Resistor_SMD:R_0402_1005Metric, symbol Device:R
- added R208: 0R 5%, Resistor_SMD:R_0402_1005Metric, symbol Device:R
- added TP12: TestPoint, TestPoint:TestPoint_Pad_D1.0mm, symbol Connector:TestPoint
- added U1: RK3568, RK3568:BGA636C65P28X28_1900X1900X168, symbol RK3568:RK3568
Connections:
- net GND: now also C362.2, C363.2
- net GMAC0_INT/PMEB_GPIO3_C0 renamed GMAC1_INT/PMEB_GPIO3_A7
- net GMAC0_MCLKINOUT renamed GMAC1_MCLKINOUT_M1
- net GMAC1_MCLKINOUT_M1: now also U1.U2 (GPIO4_C1_D)
- net GMAC0_MDC renamed GMAC1_MDC_M1
- net GMAC1_MDC_M1: now also U1.U5 (GPIO4_B6_D)
- net GMAC0_MDIO renamed GMAC1_MDIO_M1
- net GMAC1_MDIO_M1: now also U1.U4 (GPIO4_B7_D)
- net GMAC0_RSTn_GPIO3_B0 renamed GMAC1_RSTn_GPIO3_B0
- net GMAC0_RXCLK renamed GMAC1_RXCLK_M1
- net GMAC1_RXCLK_M1: now also U1.Y3 (GPIO4_A3_D)
- net GMAC0_RXD0 renamed GMAC1_RXD0_M1
- net GMAC1_RXD0_M1: now also U1.W1 (GPIO4_A7_D)
- net GMAC0_RXD1 renamed GMAC1_RXD1_M1
- net GMAC1_RXD1_M1: now also U1.V7 (GPIO4_B0_D)
- net GMAC0_RXD2 renamed GMAC1_RXD2_M1
- net GMAC1_RXD2_M1: now also U1.AA2 (GPIO4_A1_D)
- net GMAC0_RXD3 renamed GMAC1_RXD3_M1
- net GMAC1_RXD3_M1: now also U1.Y4 (GPIO4_A2_D)
- net GMAC0_RXDV_CRS renamed GMAC1_RXDV_CRS_M1
- net GMAC1_RXDV_CRS_M1: now also U1.V2 (GPIO4_B1_D)
- net GMAC0_TXCLK renamed GMAC1_TXCLK_M1
- net GMAC1_TXCLK_M1: now also R204.2
- net GMAC0_TXD0 renamed GMAC1_TXD0_M1
- net GMAC1_TXD0_M1: now also R205.2
- net GMAC0_TXD1 renamed GMAC1_TXD1_M1
- net GMAC1_TXD1_M1: now also R206.2
- net GMAC0_TXD2 renamed GMAC1_TXD2_M1
- net GMAC1_TXD2_M1: now also R202.2
- net GMAC0_TXD3 renamed GMAC1_TXD3_M1
- net GMAC1_TXD3_M1: now also R203.2
- net GMAC0_TXEN renamed GMAC1_TXEN_M1
- net GMAC1_TXEN_M1: now also R207.2
- new net: R206.1, U1.Y1 (GPIO4_A5_D)
- new net: R203.1, U1.Y5 (GPIO3_D7_D)
- new net: R202.1, U1.Y6 (GPIO3_D6_D)
- new net: R204.1, U1.AA3 (GPIO4_A0_D)
- new net: TP12.1, U1.V4 (GPIO4_B2_D)
- new net: R207.1, U1.W2 (GPIO4_A6_D)
- new net: R205.1, U1.Y2 (GPIO4_A4_D)
- new net I2C2_SCL_M1: R201.2, U1.V5 (GPIO4_B5_D)
- new net I2C2_SDA_M1: R200.2, U1.V6 (GPIO4_B4_D)
- new net MIPI_CAM0_PDN_L_GPIO3_C7: U1.AA6 (GPIO3_C7_D)
- new net MIPI_CAM0_RST_L_GPIO3_C6: U1.AC5 (GPIO3_C6_D)
- new net VCCIO6: C362.1, C363.1, R200.1, R201.1, R208.1, U1.R9 (VCCIO6), U1.U9 (VCCIO6)
- new net VCC_1V8: R208.2
- no-connect marks 0 -> 8
Other:
- note added: "Giga Phy"
- moved on the sheet: C180, C181, C182, C183, C184, C185, C186, C187, C188, C189, C190, C191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

Commit message: finished beautifying schematic
Other:
- note added: "Clock"
- note added: "Config"
- note added: "Ethernet Port"
- note added: "Ethernet Transceiver"
- note added: "Frost"
- note added: "RK3568"
- note removed: "Giga Phy"
- moved on the sheet: C177, C178, C179, C180, C181, C182, C183, C184, C185, C186, C187, C188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
